Commit message: add more models, fixed gazebo crashing bug

File: mrsl_quadrotor_description/urdf/pelican/pelican.gazebo.xacro (robot description, xacro)
@@ -2,4 +2,4 @@
 <robot name="pelican" xmlns:xacro="http://ros.org/wiki/xacro">
   <xacro:include filename="$(find mrsl_quadrotor_description)/urdf/pelican/pelican_so3.urdf.xacro" />
-  <xacro:include filename="$(find mrsl_quadrotor_description)/urdf/pelican/pelican_sensors.urdf.xacro" />
+  <xacro:include filename="$(find mrsl_quadrotor_description)/urdf/pelican/pelican_sensors.urdf.xacro"/>
 </robot>

File: mrsl_quadrotor_description/urdf/pelican/pelican_sensors.urdf.xacro (robot description, xacro)
@@ -2,12 +2,12 @@
 <robot xmlns:xacro="http://ros.org/wiki/xacro">
   <!-- Hokuyo UTM-30LX mounted upside down below the quadrotor body -->
-  <xacro:include filename="$(find mrsl_quadrotor_description)/urdf/sensors/hokuyo_utm30lx.urdf.xacro" />
+  <xacro:include filename="$(find mrsl_quadrotor_description)/urdf/sensors/hokuyo_utm30lx_with_cap.urdf.xacro" />
   <xacro:hokuyo_utm30lx name="laser" parent="base_link" ros_topic="scan" update_rate="40" ray_count="1081" min_angle="-135" max_angle="135">
-    <origin xyz="0.0 0.0 0.08" rpy="0 0 ${M_PI/4}"/>
+    <origin xyz="0.0 0.0 0.09" rpy="0 0 ${M_PI/4}"/>
   </xacro:hokuyo_utm30lx>
   <!-- Asus Xiton Live Pro -->
   <xacro:include filename="$(find mrsl_quadrotor_description)/urdf/sensors/asus_camera.urdf.xacro" />
   <xacro:asus_camera name="camera" parent="base_link">
-    <origin xyz="-0.02 0.04 0.12" rpy="${M_PI} 0 ${M_PI/4}"/>
+    <origin xyz="-0.00 0.030 0.145" rpy="${M_PI} 0 ${M_PI/4}"/>
   </xacro:asus_camera>
 </robot>

File: mrsl_quadrotor_description/urdf/sensors/asus_camera.urdf.xacro (robot description, xacro)
@@ -17,5 +17,5 @@
           <origin xyz="0 0 0" rpy="0 0 0" />
           <geometry>
-            <mesh filename="package://mrsl_models/models/sensors/asus_camera/asus_camera_simple.dae"/>
+            <mesh filename="package://mrsl_models/models/sensors/kinect/kinect.dae"/>
           </geometry>
         </visual>
@@ -23,5 +23,6 @@
           <origin xyz="0 0 0" rpy="0 0 0" />
           <geometry>
-            <box size="0.035 0.185 0.025"/>
+            <!--<box size="0.035 0.185 0.025"/>-->
+            <mesh filename="package://mrsl_models/models/sensors/kinect/kinect.stl"/>
           </geometry>
         </collision>

File: mrsl_quadrotor_description/urdf/sensors/hokuyo_utm30lx_with_cap.urdf.xacro (robot description, xacro)
@@ -7,4 +7,9 @@
         <parent link="${parent}"/>
         <child link="${name}_frame"/>
+      </joint>
+      <joint name="${name}_cap_joint" type="fixed">
+        <xacro:insert_block name="origin" />
+        <parent link="${parent}"/>
+        <child link="${name}_cap"/>
       </joint>
       <link name="${name}_frame">
@@ -26,4 +31,19 @@
             <mesh filename="package://mrsl_models/models/sensors/hokuyo_utm_30lx/utm_30lx.stl"/>
         </geometry>
+        </collision>
+      </link>
+      <link name="${name}_cap">
+        <visual>
+          <origin xyz="-0.01 0 0.027" rpy="0 0 0" />
+          <geometry>
+            <mesh filename="package://mrsl_models/models/sensors/laser_cap/laser_cap.dae"/>
+          </geometry>
+        </visual>
+        <collision>
+          <origin xyz="-0.01 0 0.027" rpy="0 0 0" />
+          <geometry>
+            <!--<box size="0.058 0.058 0.087" />-->
+            <mesh filename="package://mrsl_models/models/sensors/laser_cap/laser_cap.stl"/>
+          </geometry>
         </collision>
       </link>
