Commit message: add rotating laser model

File: mrsl_quadrotor_description/urdf/pelican/pelican_so3.urdf.xacro (robot description, xacro)
@@ -1,5 +1,4 @@
 <?xml version="1.0"?>
 <robot name="quadrotor" xmlns:xacro="http://ros.org/wiki/xacro">
-  <xacro:property name="pi" value="3.1415926535897931" />
   <xacro:property name="mass" value="0.5" />
   <xacro:property name="ixx" value="0.00264" />
@@ -23,5 +22,5 @@
         <origin xyz="0 0 0" rpy="0 0 0" />
         <geometry>
-          <mesh filename="package://mrsl_models/models/pelican/pelican.stl"/>
+          <cylinder radius="0.1" length="0.2"/>
         </geometry>
       </collision>
@@ -31,6 +30,5 @@
       <!-- Quad Dynamics Plugin -->
       <plugin name="quadrotor_propulsion" filename="libmrsl_quadrotor_propulsion.so">
-        <!--<command_topic>so3_cmd</command_topic>-->
-        <command_topic>safe_so3_cmd</command_topic>
+        <command_topic>so3_cmd</command_topic>
         <odom_topic>ground_truth/odom</odom_topic>
       </plugin>
