Commit message: add stereo camera plugin

File: mrsl_quadrotor_description/urdf/pelican/romeo/pelican_sensors.urdf.xacro (robot description, xacro)
@@ -5,4 +5,5 @@
     <origin xyz="0.0 0.0 0.09" rpy="0 0 ${M_PI/4}"/>
   </xacro:hokuyo_utm30lx>
+  <!--
   <xacro:include filename="$(find mrsl_quadrotor_description)/urdf/sensors/left_camera.urdf.xacro" />
   <xacro:camera_left name="camera_left" parent="base_link">
@@ -13,3 +14,8 @@
     <origin xyz="0.07777 -0.07777 0.145" rpy="0 0 ${M_PI/4}"/>
   </xacro:camera_right>
+-->
+ <xacro:include filename="$(find mrsl_quadrotor_description)/urdf/sensors/stereo_camera.urdf.xacro" />
+ <xacro:stereo_camera name="stereo" parent="base_link">
+   <origin xyz="0.0 0.0 0.14" rpy="0 0 ${M_PI/4}"/>
+ </xacro:stereo_camera>
 </robot>

Commit message: add texture and light source

File: mrsl_quadrotor_description/urdf/pelican/romeo/pelican_sensors.urdf.xacro (robot description, xacro)
@@ -17,5 +17,5 @@
  <xacro:include filename="$(find mrsl_quadrotor_description)/urdf/sensors/stereo_camera.urdf.xacro" />
  <xacro:stereo_camera name="stereo" parent="base_link">
-   <origin xyz="0.0 0.0 0.14" rpy="0 0 ${M_PI/4}"/>
+   <origin xyz="0.0 0.0 0.2" rpy="0 0 ${M_PI/4}"/>
  </xacro:stereo_camera>
 </robot>

Commit message: stereo_camera integrated

File: mrsl_quadrotor_description/urdf/pelican/romeo/pelican_sensors.urdf.xacro (robot description, xacro)
@@ -17,5 +17,5 @@
  <xacro:include filename="$(find mrsl_quadrotor_description)/urdf/sensors/stereo_camera.urdf.xacro" />
  <xacro:stereo_camera name="stereo" parent="base_link">
-   <origin xyz="0.0 0.0 0.2" rpy="0 0 ${M_PI/4}"/>
+   <origin xyz="0.0 0.0 0.3" rpy="0 0 ${M_PI/4}"/>
  </xacro:stereo_camera>
 </robot>

File: mrsl_quadrotor_description/urdf/pelican/romeo/pelican_so3.urdf.xacro (robot description, xacro)
@@ -56,10 +56,10 @@
         <rpyOffsets>0 0 0</rpyOffsets>
         <gaussianNoise>0</gaussianNoise>
-        <accelDrift>0.5 0.5 0.5</accelDrift>
-        <accelGaussianNoise>0.35 0.35 0.3</accelGaussianNoise>
-        <rateDrift>0.1 0.1 0.1</rateDrift>
-        <rateGaussianNoise>0.05 0.05 0.015</rateGaussianNoise>
-        <headingDrift>0.1</headingDrift>
-        <headingGaussianNoise>0.05</headingGaussianNoise>
+        <accelDrift>0.01 0.01 0.01</accelDrift>
+        <accelGaussianNoise>0.01 0.01 0.01</accelGaussianNoise>
+        <rateDrift>0.01 0.01 0.01</rateDrift>
+        <rateGaussianNoise>0.001 0.001 0.001</rateGaussianNoise>
+        <headingDrift>0.01</headingDrift>
+        <headingGaussianNoise>0.01</headingGaussianNoise>
       </plugin>
     </gazebo>

File: mrsl_quadrotor_description/urdf/sensors/stereo_camera.urdf.xacro (robot description, xacro)
@@ -5,6 +5,7 @@
   <xacro:property name="image_width" value="640" />
   <xacro:property name="image_format" value="R8G8B8" />
-  <xacro:property name="hfov" value="${M_PI/3}" />
+  <xacro:property name="hfov" value="${M_PI/2}" />
   <xacro:property name="frame_id" value="camera" />
+  <xacro:property name="focal_length" value="320" />
   <xacro:property name="hack_baseline" value="0.11" />
   <xacro:macro name="stereo_camera" params="name parent *origin">
@@ -23,5 +24,5 @@
         <origin xyz="0.0 -0.0 0" rpy="0 0 0" />
         <geometry>
-          <box size="0.1 0.05 0.025"/>
+          <box size="0.025 0.15 0.025"/>
         </geometry>
       </visual>
@@ -70,10 +71,10 @@
           <cameraInfoTopicName>camera_info</cameraInfoTopicName>
           <frameName>${frame_id}</frameName>
-          <hackBaseline>${hack_baseline}</hackBaseline>
+          <hackBaseline>${2 * hack_baseline}</hackBaseline>
           <CxPrime>${(image_width+1)/2}</CxPrime>
           <Cx>${(image_width+1)/2}</Cx>
           <Cy>${(image_height+1)/2}</Cy>
-          <!--calLength>${focal_length}</focalLength-->
-<!-- image_width / (2*tan(hfov_radian /2)) -->
+          <!--<focalLength>${focal_length}</focalLength>-->
+          <!-- image_width / (2*tan(hfov_radian /2)) -->
           <distortionK1>0.0</distortionK1>
           <distortionK2>0.0</distortionK2>

Commit message: add house environment for vision

File: mrsl_quadrotor_description/urdf/pelican/romeo/pelican_sensors.urdf.xacro (robot description, xacro)
@@ -1,21 +1,11 @@
 <?xml version="1.0"?>
 <robot xmlns:xacro="http://ros.org/wiki/xacro">
-  <xacro:include filename="$(find mrsl_quadrotor_description)/urdf/sensors/hokuyo_utm30lx_with_cap.urdf.xacro" />
-  <xacro:hokuyo_utm30lx name="laser" parent="base_link" ros_topic="laser/scan" update_rate="40" ray_count="1081" min_angle="-135" max_angle="135">
+  <xacro:include filename="$(find mrsl_quadrotor_description)/urdf/sensors/hokuyo_utm30lx.urdf.xacro" />
+  <xacro:hokuyo_utm30lx name="laser" parent="base_link" ros_topic="laser/scan" update_rate="10" ray_count="1081" min_angle="-135" max_angle="135">
     <origin xyz="0.0 0.0 0.09" rpy="0 0 ${M_PI/4}"/>
   </xacro:hokuyo_utm30lx>
-  <!--
-  <xacro:include filename="$(find mrsl_quadrotor_description)/urdf/sensors/left_camera.urdf.xacro" />
-  <xacro:camera_left name="camera_left" parent="base_link">
-    <origin xyz="-0.07777 0.07777 0.145" rpy="0 0 ${M_PI/4}"/>
-  </xacro:camera_left>
-  <xacro:include filename="$(find mrsl_quadrotor_description)/urdf/sensors/right_camera.urdf.xacro" />
-  <xacro:camera_right name="camera_right" parent="base_link">
-    <origin xyz="0.07777 -0.07777 0.145" rpy="0 0 ${M_PI/4}"/>
-  </xacro:camera_right>
--->
- <xacro:include filename="$(find mrsl_quadrotor_description)/urdf/sensors/stereo_camera.urdf.xacro" />
- <xacro:stereo_camera name="stereo" parent="base_link">
-   <origin xyz="0.0 0.0 0.3" rpy="0 0 ${M_PI/4}"/>
- </xacro:stereo_camera>
+  <xacro:include filename="$(find mrsl_quadrotor_description)/urdf/sensors/stereo_camera.urdf.xacro" />
+  <xacro:stereo_camera name="stereo" parent="base_link">
+    <origin xyz="0.0 0.0 0.3" rpy="0 0 ${M_PI/4}"/>
+  </xacro:stereo_camera>
 </robot>

File: mrsl_quadrotor_description/urdf/pelican/romeo/pelican_so3.urdf.xacro (robot description, xacro)
@@ -6,10 +6,4 @@
   <xacro:property name="iyy" value="0.00264" />
   <xacro:property name="izz" value="0.00496" />
-  <!--
-  <xacro:property name="mass" value="1.8" />
-  <xacro:property name="ixx" value="0.012" />
-  <xacro:property name="iyy" value="0.012" />
-  <xacro:property name="izz" value="0.024" />
--->
   <!-- Main quadrotor link -->
   <xacro:macro name="quadrotor_base_macro">
@@ -23,4 +17,5 @@
         <origin xyz="0 0 0" rpy="0 0 0" />
         <geometry>
+          <!--<box size="0.15 0.15 0.025"/>-->
           <mesh filename="package://mrsl_models/models/pelican/pelican.dae"/>
         </geometry>
@@ -29,4 +24,5 @@
         <origin xyz="0 0 0" rpy="0 0 0" />
         <geometry>
+          <!--<box size="0.15 0.15 0.025"/>-->
           <mesh filename="package://mrsl_models/models/pelican/pelican.stl"/>
         </geometry>

File: mrsl_quadrotor_description/urdf/sensors/stereo_camera.urdf.xacro (robot description, xacro)
@@ -9,4 +9,5 @@
   <xacro:property name="focal_length" value="320" />
   <xacro:property name="hack_baseline" value="0.11" />
+  <xacro:property name="frame_rate" value="25" />
   <xacro:macro name="stereo_camera" params="name parent *origin">
     <joint name="${name}_joint" type="fixed">
@@ -27,15 +28,9 @@
         </geometry>
       </visual>
-      <collision>
-        <origin xyz="0 0.0 0" rpy="0 0 0" />
-        <geometry>
-          <mesh filename="package://mrsl_models/models/sensors/stereo_camera/stereo_camera.stl"/>
-        </geometry>
-      </collision>
     </link>
     <!-- camera -->
     <gazebo reference="${name}_link">
       <sensor type="multicamera" name="gazebo_${name}_camera">
-        <update_rate>30.0</update_rate>
+        <update_rate>${frame_rate}</update_rate>
         <camera name="left">
           <pose>0 ${hack_baseline} 0 0 0 0</pose>
@@ -48,5 +43,5 @@
           <clip>
             <near>0.01</near>
-            <far>100</far>
+            <far>20</far>
           </clip>
         </camera>
@@ -61,10 +56,10 @@
           <clip>
             <near>0.01</near>
-            <far>100</far>
+            <far>20</far>
           </clip>
         </camera>
         <plugin name="${name}_controller" filename="libgazebo_ros_multicamera.so">
           <alwaysOn>true</alwaysOn>
-          <updateRate>30.0</updateRate>
+          <updateRate>${frame_rate}</updateRate>
           <cameraName>${name}</cameraName>
           <imageTopicName>image</imageTopicName>

Commit message: state farm demo

File: mrsl_quadrotor_description/urdf/pelican/romeo/pelican_sensors.urdf.xacro (robot description, xacro)
@@ -2,10 +2,14 @@
 <robot xmlns:xacro="http://ros.org/wiki/xacro">
   <xacro:include filename="$(find mrsl_quadrotor_description)/urdf/sensors/hokuyo_utm30lx.urdf.xacro" />
-  <xacro:hokuyo_utm30lx name="laser" parent="base_link" ros_topic="laser/scan" update_rate="10" ray_count="1081" min_angle="-135" max_angle="135">
+  <xacro:hokuyo_utm30lx name="laser" parent="base_link" ros_topic="laser/scan" update_rate="20" ray_count="1081" min_angle="-135" max_angle="135">
     <origin xyz="0.0 0.0 0.09" rpy="0 0 ${M_PI/4}"/>
   </xacro:hokuyo_utm30lx>
+  <xacro:include filename="$(find mrsl_quadrotor_description)/urdf/sensors/laser_beam.urdf.xacro" />
+  <xacro:laser_beam name="laser_beam" parent="base_link" ros_topic="laser/beam" update_rate="20" ray_count="10" min_angle="-1.25" max_angle="1.25">
+    <origin xyz="-0.05 0.05 0.09" rpy="0 ${M_PI/2} -${M_PI/4}"/>
+  </xacro:laser_beam>
   <xacro:include filename="$(find mrsl_quadrotor_description)/urdf/sensors/stereo_camera.urdf.xacro" />
   <xacro:stereo_camera name="stereo" parent="base_link">
-    <origin xyz="0.0 0.0 0.3" rpy="0 0 ${M_PI/4}"/>
+    <origin xyz="0.0 0.0 0.15" rpy="0 0 ${M_PI/4}"/>
   </xacro:stereo_camera>
 </robot>

File: mrsl_quadrotor_description/urdf/sensors/hokuyo_utm30lx.urdf.xacro (robot description, xacro)
@@ -49,5 +49,5 @@
             </scan>
             <range>
-              <min>0.3</min>
+              <min>0.1</min>
               <max>30.0</max>
               <resolution>0.01</resolution>

Commit message: add downward facing camera

File: mrsl_quadrotor_description/urdf/pelican/romeo/pelican_sensors.urdf.xacro (robot description, xacro)
@@ -13,3 +13,7 @@
     <origin xyz="0.0 0.0 0.15" rpy="0 0 ${M_PI/4}"/>
   </xacro:stereo_camera>
+  <xacro:include filename="$(find mrsl_quadrotor_description)/urdf/sensors/camera.urdf.xacro" />
+  <xacro:monocular_camera name="downward_camera" parent="base_link">
+    <origin xyz="0.1 -0.1 0.0" rpy="0 ${M_PI/2} 0"/>
+  </xacro:monocular_camera>
 </robot>

File: mrsl_quadrotor_description/urdf/sensors/camera.urdf.xacro (robot description, xacro)
@@ -2,5 +2,5 @@
 <robot xmlns:xacro="http://ros.org/wiki/xacro">
   <xacro:property name="M_PI" value="3.1415926535897931" />
-  <xacro:macro name="camera_model" params="name parent *origin">
+  <xacro:macro name="monocular_camera" params="name parent *origin">
     <joint name="${name}_joint" type="fixed">
       <xacro:insert_block name="origin" />
@@ -17,21 +17,15 @@
         <origin xyz="0.0 0.0 0" rpy="0 0 0" />
         <geometry>
-          <box size="0.1 0.05 0.025"/>
+          <box size="0.03 0.03 0.01"/>
           <!--mesh filename="package://mrsl_models/models/sensors/kinect/kinect.dae"/-->
         </geometry>
       </visual>
-      <collision>
-        <origin xyz="0 0.0 0" rpy="0 0 0" />
-        <geometry>
-          <box size="0.1 0.05 0.025"/>
-        </geometry>
-      </collision>
-    </link>
+   </link>
     <!-- camera -->
     <gazebo reference="${name}_link">
       <sensor type="camera" name="${name}">
-        <update_rate>30.0</update_rate>
+        <update_rate>5.0</update_rate>
         <camera name="head">
-          <horizontal_fov>${M_PI}/2</horizontal_fov>
+          <horizontal_fov>${M_PI/2}</horizontal_fov>
           <image>
             <width>640</width>
@@ -49,8 +43,8 @@
           </noise>
         </camera>
-        <plugin name="${name}_camera_controller" filename="libgazebo_ros_camera.so">
+        <plugin name="${name}_controller" filename="libgazebo_ros_camera.so">
           <alwaysOn>true</alwaysOn>
           <updateRate>0.0</updateRate>
-          <cameraName>camera1</cameraName>
+          <cameraName>camera</cameraName>
           <imageTopicName>image_raw</imageTopicName>
           <cameraInfoTopicName>camera_info</cameraInfoTopicName>
