Commit message: test for FLA

File: mrsl_quadrotor_description/urdf/pelican_laser_rgbd/pelican_sensors.urdf.xacro (robot description, xacro)
@@ -1,11 +1,14 @@
 <?xml version="1.0"?>
 <robot xmlns:xacro="http://ros.org/wiki/xacro">
-  <xacro:include filename="$(find mrsl_quadrotor_description)/urdf/sensors/hokuyo_utm30lx_with_cap.urdf.xacro" />
+  <!--<xacro:include filename="$(find mrsl_quadrotor_description)/urdf/sensors/hokuyo_utm30lx_with_cap.urdf.xacro" />-->
+  <xacro:include filename="$(find mrsl_quadrotor_description)/urdf/sensors/hokuyo_utm30lx.urdf.xacro" />
   <xacro:hokuyo_utm30lx name="laser" parent="base_link" ros_topic="laser/scan" update_rate="40" ray_count="1081" min_angle="-135" max_angle="135">
-    <origin xyz="0.0 0.0 0.09" rpy="0 0 ${M_PI/4}"/>
+    <origin xyz="0.0 0.0 0.2" rpy="0 0 ${M_PI/4}"/>
   </xacro:hokuyo_utm30lx>
+  <!--
   <xacro:include filename="$(find mrsl_quadrotor_description)/urdf/sensors/asus_camera.urdf.xacro" />
   <xacro:asus_camera name="camera" parent="base_link">
-    <origin xyz="-0.00 0.030 0.145" rpy="${M_PI} 0 ${M_PI/4}"/>
+    <origin xyz="0.0 0.0 0.145" rpy="${M_PI} 0 ${M_PI/4}"/>
   </xacro:asus_camera>
+-->
 </robot>

File: mrsl_quadrotor_description/urdf/sensors/asus_camera.urdf.xacro (robot description, xacro)
@@ -62,8 +62,8 @@
           <update_rate>15</update_rate>
           <camera>
-            <horizontal_fov>${62.8 * M_PI/180.0}</horizontal_fov>
+            <horizontal_fov>${90 * M_PI/180.0}</horizontal_fov>
             <image>
               <format>R8G8B8</format>
-              <width>640</width>
+              <width>752</width>
               <height>480</height>
             </image>

File: mrsl_quadrotor_description/urdf/sensors/hokuyo_utm30lx.urdf.xacro (robot description, xacro)
@@ -49,5 +49,5 @@
             </scan>
             <range>
-              <min>0.1</min>
+              <min>0.01</min>
               <max>30.0</max>
               <resolution>0.01</resolution>

File: mrsl_quadrotor_description/urdf/sensors/hokuyo_utm30lx_with_cap.urdf.xacro (robot description, xacro)
@@ -71,5 +71,5 @@
             </scan>
             <range>
-              <min>0.3</min>
+              <min>0.01</min>
               <max>30.0</max>
               <resolution>0.01</resolution>

Commit message: add pelican without frame

File: mrsl_quadrotor_description/urdf/pelican_laser_rgbd/pelican_sensors.urdf.xacro (robot description, xacro)
@@ -8,5 +8,5 @@
   <xacro:include filename="$(find mrsl_quadrotor_description)/urdf/sensors/asus_camera.urdf.xacro" />
   <xacro:asus_camera name="camera" parent="base_link">
-    <origin xyz="0.1 0.1 0.0" rpy="${M_PI} 0 ${M_PI/4}"/>
+    <origin xyz="0.11 0.11 0.0" rpy="${M_PI} 0 ${M_PI/4}"/>
   </xacro:asus_camera>
 </robot>

File: mrsl_quadrotor_description/urdf/pelican_laser_rgbd/pelican_so3.urdf.xacro (robot description, xacro)
@@ -17,5 +17,5 @@
         <origin xyz="0 0 0" rpy="0 0 0" />
         <geometry>
-          <mesh filename="package://mrsl_models/models/pelican/pelican.dae"/>
+          <mesh filename="package://mrsl_models/models/pelican/pelican_without_frame.dae"/>
         </geometry>
       </visual>
