Commit message: fix some bugs

File: mrsl_quadrotor_description/urdf/hummingbird_rgbd/hummingbird_so3.urdf.xacro (robot description, xacro)
@@ -16,5 +16,5 @@
       </inertial>
       <visual>
-        <origin xyz="0 0 0" rpy="0 0 0" />
+        <origin xyz="0 0 0" rpy="0 0 0.0"/>
         <geometry>
           <mesh filename="package://mrsl_models/models/hummingbird/hummingbird.dae"/>
