Commit message: change some params for sensors, add hummingbird rgbd model

File: mrsl_quadrotor_description/urdf/hummingbird_rgbd/hummingbird_sensors.urdf.xacro (robot description, xacro)
@@ -2,10 +2,12 @@
 <robot xmlns:xacro="http://ros.org/wiki/xacro">
   <xacro:include filename="$(find mrsl_quadrotor_description)/urdf/sensors/asus_camera.urdf.xacro" />
-  <xacro:asus_camera name="camera_left" parent="base_link">
-    <origin xyz="0.0 0.1 0.2" rpy="${M_PI} 0 ${M_PI/2}"/>
+  <xacro:asus_camera name="camera" parent="base_link">
+    <origin xyz="0.02 0.02 0.16" rpy="${M_PI} 0 ${M_PI/4}"/>
   </xacro:asus_camera>
+  <!--
   <xacro:include filename="$(find mrsl_quadrotor_description)/urdf/sensors/asus_camera.urdf.xacro" />
   <xacro:asus_camera name="camera_right" parent="base_link">
-    <origin xyz="0.1 0.0 0.2" rpy="${M_PI} 0 0"/>
+    <origin xyz="0.06 0.0 0.16" rpy="${M_PI} 0 0"/>
   </xacro:asus_camera>
+-->
 </robot>

File: mrsl_quadrotor_description/urdf/hummingbird_rgbd/hummingbird_so3.urdf.xacro (robot description, xacro)
@@ -10,4 +10,5 @@
     <link name="base_link">
       <inertial>
+        <!--mass value="1.477" /-->
         <mass value="${mass}"/>
         <origin xyz="0 0 0" />
@@ -17,11 +18,12 @@
         <origin xyz="0 0 0" rpy="0 0 0" />
         <geometry>
-          <mesh filename="package://mrsl_models/models/pelican/pelican.dae"/>
+          <mesh filename="package://mrsl_models/models/hummingbird/hummingbird.dae"/>
         </geometry>
       </visual>
       <collision>
-        <origin xyz="0 0 0" rpy="0 0 0" />
+        <origin xyz="0 0 0" rpy="0 0 0.7854" />
         <geometry>
-          <mesh filename="package://mrsl_models/models/pelican/pelican.stl"/>
+          <!--mesh filename="package://mrsl_models/models/hummingbird/hummingbird.stl"/-->
+          <box size="0.3 0.3 0.2" />
         </geometry>
       </collision>
@@ -30,7 +32,7 @@
     <gazebo>
       <!-- Quad Dynamics Plugin -->
-      <plugin name="quadrotor_propulsion" filename="libmrsl_quadrotor_propulsion.so">
+      <plugin name="test" filename="libmrsl_quadrotor_propulsion.so">
         <command_topic>so3_cmd</command_topic>
-        <odom_topic>ground_truth/odom</odom_topic>
+        <!--<odom_topic>ground_truth/odom</odom_topic>-->
       </plugin>
       <!-- Quad Ground Truth Plugin -->
@@ -47,6 +49,6 @@
         <bodyName>base_link</bodyName>
         <topicName>raw_imu</topicName>
-        <rpyOffsets>0 0 0</rpyOffsets>
-        <gaussianNoise>0</gaussianNoise>
+        <rpyOffsets>0 0 0</rpyOffsets> <!-- deprecated -->
+        <gaussianNoise>0</gaussianNoise>  <!-- deprecated -->
         <accelDrift>0.5 0.5 0.5</accelDrift>
         <accelGaussianNoise>0.35 0.35 0.3</accelGaussianNoise>

File: mrsl_quadrotor_description/urdf/sensors/asus_camera.urdf.xacro (robot description, xacro)
@@ -17,5 +17,5 @@
           <origin xyz="0 0 0" rpy="0 0 0" />
           <geometry>
-            <mesh filename="package://mrsl_models/models/sensors/kinect/kinect.dae"/>
+            <mesh filename="package://mrsl_models/models/sensors/asus_camera/asus_camera.dae"/>
           </geometry>
         </visual>
@@ -24,5 +24,5 @@
           <geometry>
             <!--<box size="0.035 0.185 0.025"/>-->
-            <mesh filename="package://mrsl_models/models/sensors/kinect/kinect.stl"/>
+            <mesh filename="package://mrsl_models/models/sensors/asus_camera/asus_camera.stl"/>
           </geometry>
         </collision>

Commit message: add utils, and several maps and models

File: mrsl_quadrotor_description/urdf/hummingbird_rgbd/hummingbird_sensors.urdf.xacro (robot description, xacro)
@@ -1,7 +1,7 @@
 <?xml version="1.0"?>
 <robot xmlns:xacro="http://ros.org/wiki/xacro">
-  <xacro:include filename="$(find mrsl_quadrotor_description)/urdf/sensors/asus_camera.urdf.xacro" />
+  <xacro:include filename="$(find mrsl_quadrotor_description)/urdf/sensors/asus_camera_60.urdf.xacro" />
   <xacro:asus_camera name="camera" parent="base_link">
-    <origin xyz="0.02 0.02 0.16" rpy="${M_PI} 0 ${M_PI/4}"/>
+    <origin xyz="0.1 0.1 0.0" rpy="${M_PI} 0 ${M_PI/4}"/>
   </xacro:asus_camera>
   <!--

File: mrsl_quadrotor_description/urdf/pelican_laser_rgbd/pelican_sensors.urdf.xacro (robot description, xacro)
@@ -4,11 +4,9 @@
   <xacro:include filename="$(find mrsl_quadrotor_description)/urdf/sensors/hokuyo_utm30lx.urdf.xacro" />
   <xacro:hokuyo_utm30lx name="laser" parent="base_link" ros_topic="laser/scan" update_rate="40" ray_count="1081" min_angle="-135" max_angle="135">
-    <origin xyz="0.0 0.0 0.2" rpy="0 0 ${M_PI/4}"/>
+    <origin xyz="0.0 0.0 0.1" rpy="0 0 ${M_PI/4}"/>
   </xacro:hokuyo_utm30lx>
-  <!--
   <xacro:include filename="$(find mrsl_quadrotor_description)/urdf/sensors/asus_camera.urdf.xacro" />
   <xacro:asus_camera name="camera" parent="base_link">
-    <origin xyz="0.0 0.0 0.145" rpy="${M_PI} 0 ${M_PI/4}"/>
+    <origin xyz="0.1 0.1 0.0" rpy="${M_PI} 0 ${M_PI/4}"/>
   </xacro:asus_camera>
--->
 </robot>

File: mrsl_quadrotor_description/urdf/sensors/hokuyo_utm30lx.urdf.xacro (robot description, xacro)
@@ -59,5 +59,5 @@
             <updateRate>${update_rate}</updateRate>
             <topicName>${ros_topic}</topicName>
-            <frameName>${name}_frame</frameName>
+            <frameName>${name}</frameName>
           </plugin>
         </sensor>
