Commit message: add stereo model

File: mrsl_quadrotor_description/urdf/hummingbird/hummingbird.gazebo.xacro (robot description, xacro)
@@ -2,4 +2,3 @@
 <robot name="hummingbird" xmlns:xacro="http://ros.org/wiki/xacro">
   <xacro:include filename="$(find mrsl_quadrotor_description)/urdf/hummingbird/hummingbird_so3.urdf.xacro" />
-  <!--xacro:include filename="$(find mrsl_quadrotor_description)/urdf/hummingbird/hummingbird_sensors.urdf.xacro" /-->
 </robot>

File: mrsl_quadrotor_description/urdf/hummingbird_rgbd/hummingbird_rgbd.gazebo.xacro (robot description, xacro)
@@ -1,6 +1,5 @@
 <?xml version="1.0"?>
 <robot name="pelican" xmlns:xacro="http://ros.org/wiki/xacro">
-  <!--xacro:include filename="$(find mrsl_quadrotor_description)/urdf/pelican_rgbd/pelican_so3.urdf.xacro" /-->
-  <xacro:include filename="$(find mrsl_quadrotor_description)/urdf/hummingbird_rgbd/hummingbird_so3.urdf.xacro" />
-  <xacro:include filename="$(find mrsl_quadrotor_description)/urdf/hummingbird_rgbd/hummingbird_sensors.urdf.xacro"/>
+  <xacro:include filename="$(find mrsl_quadrotor_description)/urdf/hummingbird/hummingbird_so3.urdf.xacro" />
+  <xacro:include filename="$(find mrsl_quadrotor_description)/urdf/hummingbird_rgbd/sensors.urdf.xacro"/>
 </robot>

File: mrsl_quadrotor_description/urdf/pelican/pelican.gazebo.xacro (robot description, xacro)
@@ -2,4 +2,3 @@
 <robot name="pelican" xmlns:xacro="http://ros.org/wiki/xacro">
   <xacro:include filename="$(find mrsl_quadrotor_description)/urdf/pelican/pelican_so3.urdf.xacro" />
-  <xacro:include filename="$(find mrsl_quadrotor_description)/urdf/pelican_laser_rgbd/sensors.urdf.xacro"/>
 </robot>

File: mrsl_quadrotor_description/urdf/pelican_laser_stereo/pelican_laser_stereo.gazebo.xacro (robot description, xacro)
@@ -2,4 +2,4 @@
 <robot name="pelican" xmlns:xacro="http://ros.org/wiki/xacro">
   <xacro:include filename="$(find mrsl_quadrotor_description)/urdf/pelican/pelican_so3.urdf.xacro" />
-  <xacro:include filename="$(find mrsl_quadrotor_description)/urdf/pelican_laser_rgbd/sensors.urdf.xacro"/>
+  <xacro:include filename="$(find mrsl_quadrotor_description)/urdf/pelican_laser_stereo/sensors.urdf.xacro"/>
 </robot>

File: mrsl_quadrotor_description/urdf/sensors/stereo_camera.urdf.xacro (robot description, xacro)
@@ -8,6 +8,6 @@
   <xacro:property name="frame_id" value="camera" />
   <xacro:property name="focal_length" value="320" />
-  <xacro:property name="hack_baseline" value="0.11" />
-  <xacro:property name="frame_rate" value="25" />
+  <xacro:property name="hack_baseline" value="0.10" />
+  <xacro:property name="frame_rate" value="15" />
   <xacro:macro name="stereo_camera" params="name parent *origin">
     <joint name="${name}_joint" type="fixed">
@@ -42,5 +42,5 @@
           </image>
           <clip>
-            <near>0.01</near>
+            <near>0.1</near>
             <far>20</far>
           </clip>
@@ -55,5 +55,5 @@
           </image>
           <clip>
-            <near>0.01</near>
+            <near>0.1</near>
             <far>20</far>
           </clip>
@@ -63,5 +63,5 @@
           <updateRate>${frame_rate}</updateRate>
           <cameraName>${name}</cameraName>
-          <imageTopicName>image</imageTopicName>
+          <imageTopicName>image_raw</imageTopicName>
           <cameraInfoTopicName>camera_info</cameraInfoTopicName>
           <frameName>${frame_id}</frameName>
