Commit message: fix pelican bug

File: mrsl_quadrotor_description/urdf/hummingbird/hummingbird_so3.urdf.xacro (robot description, xacro)
@@ -19,5 +19,4 @@
         <geometry>
           <mesh filename="package://mrsl_models/models/hummingbird/hummingbird.dae"/>
-          <!--mesh filename="package://mrsl_models/models/quadrotor/quadrotor.dae"/-->
         </geometry>
       </visual>

File: mrsl_quadrotor_description/urdf/pelican/pelican.gazebo.xacro (robot description, xacro)
@@ -2,4 +2,4 @@
 <robot name="pelican" xmlns:xacro="http://ros.org/wiki/xacro">
   <xacro:include filename="$(find mrsl_quadrotor_description)/urdf/pelican/pelican_so3.urdf.xacro" />
-  <xacro:include filename="$(find mrsl_quadrotor_description)/urdf/pelican/pelican_sensors.urdf.xacro"/>
+  <!--xacro:include filename="$(find mrsl_quadrotor_description)/urdf/pelican/pelican_sensors.urdf.xacro"/-->
 </robot>

File: mrsl_quadrotor_description/urdf/pelican/pelican_sensors.urdf.xacro (robot description, xacro)
@@ -1,10 +1,8 @@
 <?xml version="1.0"?>
 <robot xmlns:xacro="http://ros.org/wiki/xacro">
-  <!-- Hokuyo UTM-30LX mounted upside down below the quadrotor body -->
   <xacro:include filename="$(find mrsl_quadrotor_description)/urdf/sensors/hokuyo_utm30lx_with_cap.urdf.xacro" />
   <xacro:hokuyo_utm30lx name="laser" parent="base_link" ros_topic="scan" update_rate="40" ray_count="1081" min_angle="-135" max_angle="135">
     <origin xyz="0.0 0.0 0.09" rpy="0 0 ${M_PI/4}"/>
   </xacro:hokuyo_utm30lx>
-  <!-- Asus Xiton Live Pro -->
   <xacro:include filename="$(find mrsl_quadrotor_description)/urdf/sensors/asus_camera.urdf.xacro" />
   <xacro:asus_camera name="camera" parent="base_link">

File: mrsl_quadrotor_description/urdf/pelican/pelican_so3.urdf.xacro (robot description, xacro)
@@ -2,13 +2,18 @@
 <robot name="quadrotor" xmlns:xacro="http://ros.org/wiki/xacro">
   <xacro:property name="pi" value="3.1415926535897931" />
-  <xacro:property name="mass" value="1.815" />
+  <xacro:property name="mass" value="0.5" />
+  <xacro:property name="ixx" value="0.00264" />
+  <xacro:property name="iyy" value="0.00264" />
+  <xacro:property name="izz" value="0.00496" />
+  <!--
+  <xacro:property name="mass" value="1.8" />
   <xacro:property name="ixx" value="0.012" />
   <xacro:property name="iyy" value="0.012" />
   <xacro:property name="izz" value="0.024" />
+-->
   <!-- Main quadrotor link -->
   <xacro:macro name="quadrotor_base_macro">
     <link name="base_link">
       <inertial>
-        <!--mass value="1.477" /-->
         <mass value="${mass}"/>
         <origin xyz="0 0 0" />

File: mrsl_quadrotor_description/urdf/sensors/hokuyo_utm30lx_with_cap.urdf.xacro (robot description, xacro)
@@ -35,4 +35,6 @@
       <link name="${name}_cap">
         <visual>
+          <mass value="0.000" />
+          <inertia ixx="0" ixy="0" ixz="0" iyy="0" iyz="0" izz="0" />
           <origin xyz="-0.01 0 0.027" rpy="0 0 0" />
           <geometry>

Commit message: latest simulation for FLA, update README.md

File: mrsl_quadrotor_description/urdf/hummingbird/hummingbird_so3.urdf.xacro (robot description, xacro)
@@ -43,19 +43,5 @@
         <frameName>world</frameName>
       </plugin>
-      <!-- Quad Imu Plugin -->
-      <plugin name="quadrotor_imu_sim" filename="libhector_gazebo_ros_imu.so">
-        <updateRate>100.0</updateRate>
-        <bodyName>base_link</bodyName>
-        <topicName>raw_imu</topicName>
-        <rpyOffsets>0 0 0</rpyOffsets> <!-- deprecated -->
-        <gaussianNoise>0</gaussianNoise>  <!-- deprecated -->
-        <accelDrift>0.5 0.5 0.5</accelDrift>
-        <accelGaussianNoise>0.35 0.35 0.3</accelGaussianNoise>
-        <rateDrift>0.1 0.1 0.1</rateDrift>
-        <rateGaussianNoise>0.05 0.05 0.015</rateGaussianNoise>
-        <headingDrift>0.1</headingDrift>
-        <headingGaussianNoise>0.05</headingGaussianNoise>
-      </plugin>
-    </gazebo>
+      </gazebo>
   </xacro:macro>
   <xacro:quadrotor_base_macro/>

File: mrsl_quadrotor_description/urdf/pelican/pelican_so3.urdf.xacro (robot description, xacro)
@@ -22,5 +22,5 @@
         <origin xyz="0 0 0" rpy="0 0 0" />
         <geometry>
-          <cylinder radius="0.1" length="0.2"/>
+          <cylinder radius="0.05" length="0.1"/>
         </geometry>
       </collision>
@@ -41,19 +41,5 @@
         <frameName>world</frameName>
       </plugin>
-      <!-- Quad Imu Plugin -->
-      <plugin name="quadrotor_imu_sim" filename="libhector_gazebo_ros_imu.so">
-        <updateRate>100.0</updateRate>
-        <bodyName>base_link</bodyName>
-        <topicName>raw_imu</topicName>
-        <rpyOffsets>0 0 0</rpyOffsets>
-        <gaussianNoise>0</gaussianNoise>
-        <accelDrift>0.5 0.5 0.5</accelDrift>
-        <accelGaussianNoise>0.35 0.35 0.3</accelGaussianNoise>
-        <rateDrift>0.1 0.1 0.1</rateDrift>
-        <rateGaussianNoise>0.05 0.05 0.015</rateGaussianNoise>
-        <headingDrift>0.1</headingDrift>
-        <headingGaussianNoise>0.05</headingGaussianNoise>
-      </plugin>
-    </gazebo>
+     </gazebo>
   </xacro:macro>
   <xacro:quadrotor_base_macro/>

File: mrsl_quadrotor_description/urdf/pelican_laser/sensors.urdf.xacro (robot description, xacro)
@@ -4,5 +4,5 @@
   <xacro:include filename="$(find mrsl_quadrotor_description)/urdf/sensors/hokuyo_utm30lx.urdf.xacro" />
   <xacro:hokuyo_utm30lx name="laser" parent="base_link" ros_topic="laser/scan" update_rate="40" ray_count="1081" min_angle="-135" max_angle="135">
-    <origin xyz="0.1 0.1 0.0" rpy="0 0 ${M_PI/4}"/>
+    <origin xyz="0.0 0.0 0.2" rpy="0 0 ${M_PI/4}"/>
   </xacro:hokuyo_utm30lx>
 </robot>

File: mrsl_quadrotor_description/urdf/pelican_laser_rgbd/sensors.urdf.xacro (robot description, xacro)
@@ -4,5 +4,5 @@
   <xacro:include filename="$(find mrsl_quadrotor_description)/urdf/sensors/hokuyo_utm30lx.urdf.xacro" />
   <xacro:hokuyo_utm30lx name="laser" parent="base_link" ros_topic="laser/scan" update_rate="40" ray_count="1081" min_angle="-135" max_angle="135">
-    <origin xyz="0.0 0.0 0.1" rpy="0 0 ${M_PI/4}"/>
+    <origin xyz="0.0 0.0 0.2" rpy="0 0 ${M_PI/4}"/>
   </xacro:hokuyo_utm30lx>
   <xacro:include filename="$(find mrsl_quadrotor_description)/urdf/sensors/asus_camera.urdf.xacro" />

File: mrsl_quadrotor_description/urdf/sensors/camera.urdf.xacro (robot description, xacro)
@@ -12,5 +12,5 @@
         <mass value="0.000001" />
         <origin xyz="0 0 0" rpy="0 0 0" />
-        <inertia ixx="5.8083e-4" ixy="0" ixz="0" iyy="3.0833e-5" iyz="0" izz="5.9083e-4" />
+        <inertia ixx="1e-6" ixy="0" ixz="0" iyy="1e-6" iyz="0" izz="1e-6" />
       </inertial>
       <visual>
@@ -18,5 +18,4 @@
         <geometry>
           <box size="0.03 0.03 0.01"/>
-          <!--mesh filename="package://mrsl_models/models/sensors/kinect/kinect.dae"/-->
         </geometry>
       </visual>
@@ -46,5 +45,5 @@
           <alwaysOn>true</alwaysOn>
           <updateRate>0.0</updateRate>
-          <cameraName>camera</cameraName>
+          <cameraName>${name}</cameraName>
           <imageTopicName>image_raw</imageTopicName>
           <cameraInfoTopicName>camera_info</cameraInfoTopicName>

File: mrsl_quadrotor_description/urdf/sensors/hokuyo_utm30lx.urdf.xacro (robot description, xacro)
@@ -1,54 +1,101 @@
 <?xml version="1.0"?>
 <robot xmlns:xacro="http://ros.org/wiki/xacro">
-  <xacro:property name="M_PI" value="3.1415926535897931" />
-  <xacro:macro name="hokuyo_utm30lx" params="name parent *origin ros_topic update_rate ray_count min_angle max_angle">
-    <link name="${name}_frame">
-      <inertial>
-        <mass value="0.001" />
-        <origin xyz="0 0 0" rpy="0 0 0" />
-        <inertia ixx="2.632e-4" ixy="0" ixz="0" iyy="2.632e-4" iyz="0" izz="1.62e-4" />
-      </inertial>
-      <visual>
-        <origin xyz="0 0 0" rpy="0 0 0" />
-        <geometry>
-          <mesh filename="package://mrsl_models/models/sensors/hokuyo_utm_30lx/utm_30lx.dae"/>
+    <xacro:property name="M_PI" value="3.1415926535897931" />
+    <xacro:macro name="hokuyo_utm30lx_model" params="name parent *origin">
+      <joint name="${name}_joint" type="fixed">
+        <xacro:insert_block name="origin" />
+        <parent link="${parent}"/>
+        <child link="${name}_frame"/>
+      </joint>
+      <link name="${name}_frame">
+        <inertial>
+          <mass value="0.000" />
+          <origin xyz="0 0 0" rpy="0 0 0" />
+          <inertia ixx="2.632e-4" ixy="0" ixz="0" iyy="2.632e-4" iyz="0" izz="1.62e-4" />
+        </inertial>
+        <visual>
+          <origin xyz="0 0 0.0" rpy="0 0 0" />
+          <geometry>
+            <mesh filename="package://mrsl_models/models/sensors/hokuyo_utm_30lx/utm_30lx.dae"/>
         </geometry>
-      </visual>
-   </link>
-    <joint name="${name}_joint" type="fixed">
-      <xacro:insert_block name="origin" />
-      <parent link="${parent}"/>
-      <child link="${name}_frame"/>
-    </joint>
-    <gazebo reference="${name}_frame">
-      <sensor type="ray" name="${name}">
-        <always_on>true</always_on>
-        <update_rate>${update_rate}</update_rate>
-        <pose>0 0 0 0 0 0</pose>
-        <visualize>true</visualize>
-        <ray>
-          <scan>
-            <horizontal>
-              <samples>${ray_count}</samples>
-              <resolution>1</resolution>
-              <min_angle>${min_angle * M_PI/180}</min_angle>
-              <max_angle>${max_angle * M_PI/180}</max_angle>
-            </horizontal>
-          </scan>
-          <range>
-            <min>0.1</min>
-            <max>30.0</max>
-            <resolution>0.01</resolution>
-          </range>
-        </ray>
-        <plugin name="gazebo_ros_${name}_controller" filename="libgazebo_ros_laser.so">
-          <gaussianNoise>0.005</gaussianNoise>
-          <alwaysOn>true</alwaysOn>
-          <updateRate>${update_rate}</updateRate>
-          <topicName>${ros_topic}</topicName>
-          <frameName>${name}_frame</frameName>
-        </plugin>
-      </sensor>
-    </gazebo>
-  </xacro:macro>
+        </visual>
+        <collision>
+          <origin xyz="0 0 0.0" rpy="0 0 0" />
+          <geometry>
+            <!--<box size="0.058 0.058 0.087" />-->
+            <mesh filename="package://mrsl_models/models/sensors/hokuyo_utm_30lx/utm_30lx.stl"/>
+        </geometry>
+        </collision>
+      </link>
+    </xacro:macro>
+    <xacro:macro name="hokuyo_utm30lx" params="name parent *origin ros_topic update_rate ray_count min_angle max_angle">
+      <xacro:hokuyo_utm30lx_model name="${name}" parent="${parent}">
+        <xacro:insert_block name="origin" />
+      </xacro:hokuyo_utm30lx_model>
+      <gazebo reference="${name}_frame">
+        <sensor type="ray" name="${name}">
+          <always_on>true</always_on>
+          <update_rate>${update_rate}</update_rate>
+          <pose>0 0 0 0 0 0</pose>
+          <visualize>false</visualize>
+          <ray>
+            <scan>
+              <horizontal>
+                <samples>${ray_count}</samples>
+                <resolution>1</resolution>
+                <min_angle>${min_angle * M_PI/180}</min_angle>
+                <max_angle>${max_angle * M_PI/180}</max_angle>
+              </horizontal>
+            </scan>
+            <range>
+              <min>0.1</min>
+              <max>30.0</max>
+              <resolution>0.01</resolution>
+            </range>
+          </ray>
+          <plugin name="gazebo_ros_${name}_controller" filename="libgazebo_ros_laser.so">
+            <gaussianNoise>0.005</gaussianNoise>
+            <alwaysOn>true</alwaysOn>
+            <updateRate>${update_rate}</updateRate>
+            <topicName>${ros_topic}</topicName>
+            <frameName>${name}</frameName>
+          </plugin>
+        </sensor>
+      </gazebo>
+    </xacro:macro>
+    <xacro:macro name="hokuyo_utm30lx_gpu" params="name parent *origin ros_topic update_rate ray_count min_angle max_angle">
+      <xacro:hokuyo_utm30lx_model name="${name}" parent="${parent}">
+        <xacro:insert_block name="origin" />
+      </xacro:hokuyo_utm30lx_model>
+      <gazebo reference="${name}_frame">
+        <sensor type="gpu_ray" name="${name}">
+          <always_on>true</always_on>
+          <update_rate>${update_rate}</update_rate>
+          <pose>0 0 0 0 0 0</pose>
+          <visualize>false</visualize>
+          <ray>
+            <scan>
+              <horizontal>
+                <samples>${ray_count}</samples>
+                <resolution>1</resolution>
+                <min_angle>${min_angle * M_PI/180}</min_angle>
+                <max_angle>${max_angle * M_PI/180}</max_angle>
+              </horizontal>
+            </scan>
+            <range>
+              <min>0.3</min>
+              <max>30.0</max>
+              <resolution>0.01</resolution>
+            </range>
+          </ray>
+          <plugin name="gazebo_ros_${name}_controller" filename="libgazebo_ros_gpu_laser.so">
+            <gaussianNoise>0.005</gaussianNoise>
+            <alwaysOn>true</alwaysOn>
+            <updateRate>${update_rate}</updateRate>
+            <topicName>${ros_topic}</topicName>
+            <frameName>${name}_frame</frameName>
+          </plugin>
+        </sensor>
+      </gazebo>
+    </xacro:macro>
 </robot>

File: mrsl_quadrotor_description/urdf/sensors/hokuyo_utm30lx_rotate.urdf.xacro (robot description, xacro)
@@ -3,5 +3,5 @@
   <xacro:property name="M_PI" value="3.1415926535897931" />
   <xacro:macro name="hokuyo_utm30lx" params="name parent *origin ros_topic update_rate ray_count min_angle max_angle">
-    <link name="${name}_frame">
+    <link name="${name}">
       <inertial>
         <mass value="0.001" />
@@ -19,15 +19,15 @@
       <xacro:insert_block name="origin" />
       <parent link="${parent}"/>
-      <child link="${name}_frame"/>
+      <child link="${name}"/>
       <axis xyz="0 1 0" rpy="0 0 0" />
       <limit effort="100" velocity="10"/>
       <joint_properties damping="0.0" friction="0.0"/>
     </joint>
-    <gazebo reference="${name}_frame">
+    <gazebo reference="${name}">
       <sensor type="ray" name="${name}">
         <always_on>true</always_on>
         <update_rate>${update_rate}</update_rate>
         <pose>0 0 0 0 0 0</pose>
-        <visualize>true</visualize>
+        <visualize>false</visualize>
         <ray>
           <scan>
@@ -50,5 +50,5 @@
           <updateRate>${update_rate}</updateRate>
           <topicName>${ros_topic}</topicName>
-          <frameName>${name}_frame</frameName>
+          <frameName>${name}</frameName>
         </plugin>
       </sensor>
