Commit message: add fla_warehouse2

File: mrsl_quadrotor_description/urdf/sensors/hokuyo_utm30lx_rotate.urdf.xacro (robot description, xacro)
@@ -5,7 +5,7 @@
     <link name="${name}_frame">
       <inertial>
-        <mass value="0.010" />
+        <mass value="0.001" />
         <origin xyz="0 0 0" rpy="0 0 0" />
-        <inertia ixx="2.632e-6" ixy="0" ixz="0" iyy="2.632e-6" iyz="0" izz="1.62e-6" />
+        <inertia ixx="2.632e-4" ixy="0" ixz="0" iyy="2.632e-4" iyz="0" izz="1.62e-4" />
       </inertial>
       <visual>
@@ -29,5 +29,5 @@
         <update_rate>${update_rate}</update_rate>
         <pose>0 0 0 0 0 0</pose>
-        <visualize>false</visualize>
+        <visualize>true</visualize>
         <ray>
           <scan>
