Commit message: fix ovc link names

File: mrsl_quadrotor_description/urdf/sensors/ovc3.urdf.xacro (robot description, xacro)
@@ -6,5 +6,5 @@
   <xacro:property name="image_format" value="L8" />
   <xacro:property name="hfov" value="${M_PI/2}" />
-  <xacro:property name="frame_id" value="camera" />
+  <xacro:property name="frame_id" value="ovc_camera_link_optical" />
   <xacro:property name="focal_length" value="320" />
   <xacro:property name="hack_baseline" value="0.06" />
@@ -29,16 +29,16 @@
       </visual>
     </link>
-    <joint name="${name}_depth_joint" type="fixed">
+    <joint name="${name}_camera_joint" type="fixed">
         <origin xyz="0.002 0.06 -0.005" rpy="0 0 0" />
         <parent link="${name}_link" />
-        <child link="${name}_depth_frame"/>
+        <child link="${name}_camera_frame"/>
       </joint>
-      <link name="${name}_depth_frame"/>
-      <joint name="${name}_depth_optical_joint" type="fixed">
+      <link name="${name}_camera_frame"/>
+      <joint name="${name}_camera_optical_joint" type="fixed">
         <origin xyz="0 0 0" rpy="${-M_PI/2} 0.0 ${-M_PI/2}" />
-        <parent link="${name}_depth_frame" />
-        <child link="${name}_depth_optical_frame"/>
+        <parent link="${name}_camera_frame" />
+        <child link="${name}_camera_optical_frame"/>
       </joint>
-      <link name="${name}_depth_optical_frame"/>
+      <link name="${name}_camera_optical_frame"/>
     <!-- camera -->
     <gazebo reference="${name}_link">

File: mrsl_quadrotor_description/urdf/sensors/ovc3_extcam.urdf.xacro (robot description, xacro)
@@ -6,5 +6,5 @@
   <xacro:property name="image_format" value="L8" />
   <xacro:property name="hfov" value="${M_PI/2}" />
-  <xacro:property name="frame_id" value="camera" />
+  <xacro:property name="frame_id" value="ovc_camera_link_optical" />
   <xacro:property name="focal_length" value="320" />
   <xacro:property name="hack_baseline" value="0.06" />
@@ -29,16 +29,16 @@
       </visual>
     </link>
-    <joint name="${name}_depth_joint" type="fixed">
+    <joint name="${name}_camera_joint" type="fixed">
         <origin xyz="0.002 0.06 -0.004" rpy="0 0 0" />
         <parent link="${name}_link" />
-        <child link="${name}_depth_frame"/>
+        <child link="${name}_camera_frame"/>
       </joint>
-      <link name="${name}_depth_frame"/>
-      <joint name="${name}_depth_optical_joint" type="fixed">
+      <link name="${name}_camera_frame"/>
+      <joint name="${name}_camera_optical_joint" type="fixed">
         <origin xyz="0 0 0" rpy="${-M_PI/2} 0.0 ${-M_PI/2}" />
-        <parent link="${name}_depth_frame" />
-        <child link="${name}_depth_optical_frame"/>
+        <parent link="${name}_camera_frame" />
+        <child link="${name}_camera_optical_frame"/>
       </joint>
-      <link name="${name}_depth_optical_frame"/>
+      <link name="${name}_camera_optical_frame"/>
     <!-- camera -->
     <gazebo reference="${name}_link">
