Commit message: add fla platform rgbd range

File: mrsl_quadrotor_description/urdf/sensors/range_beam.urdf.xacro (robot description, xacro)
@@ -17,5 +17,4 @@
           <origin xyz="0 0 0" rpy="0 ${M_PI/2} 0" />
           <geometry>
-            <!--<box size="0.058 0.058 0.087" />-->
             <cylinder radius="0.01" length="0.1"/>
        </geometry>

Commit message: LidarLite URDF removed

File: mrsl_quadrotor_description/urdf/sensors/range_beam.urdf.xacro (robot description, xacro)
@@ -6,7 +6,7 @@
         <xacro:insert_block name="origin" />
         <parent link="${parent}"/>
-        <child link="${name}_frame"/>
+        <child link="${name}"/>
       </joint>
-      <link name="${name}_frame">
+      <link name="${name}">
         <inertial>
           <mass value="0.000" />
@@ -26,5 +26,5 @@
         <xacro:insert_block name="origin" />
       </xacro:range_beam_model>
-      <gazebo reference="${name}_frame">
+      <gazebo reference="${name}">
         <sensor type="ray" name="${name}">
           <always_on>true</always_on>

Commit message: Falcon4 and OVC3 components (#9)
* Falcon4 and OVC3 components added

* Falcon4 added to README.md

* Falcon4 orientation updated

* OVC3 tf updated

* CAD Models Updated

* LidarLite URDF removed

* fix ovc link names

Co-authored-by: Dinesh Thakur <tdinesh@seas.upenn.edu>

File: mrsl_quadrotor_description/urdf/sensors/range_beam.urdf.xacro (robot description, xacro)
@@ -6,7 +6,7 @@
         <xacro:insert_block name="origin" />
         <parent link="${parent}"/>
-        <child link="${name}_frame"/>
+        <child link="${name}"/>
       </joint>
-      <link name="${name}_frame">
+      <link name="${name}">
         <inertial>
           <mass value="0.000" />
@@ -17,5 +17,5 @@
           <origin xyz="0 0 0" rpy="0 ${M_PI/2} 0" />
           <geometry>
-            <cylinder radius="0.01" length="0.1"/>
+            <cylinder radius="0.01" length="0.01"/>
        </geometry>
         </visual>
@@ -26,5 +26,5 @@
         <xacro:insert_block name="origin" />
       </xacro:range_beam_model>
-      <gazebo reference="${name}_frame">
+      <gazebo reference="${name}">
         <sensor type="ray" name="${name}">
           <always_on>true</always_on>
