Commit message: add fla_warehouse2

File: mrsl_quadrotor_description/urdf/pelican_laser/sensors.urdf.xacro (robot description, xacro)
@@ -4,5 +4,5 @@
   <xacro:include filename="$(find mrsl_quadrotor_description)/urdf/sensors/hokuyo_utm30lx.urdf.xacro" />
   <xacro:hokuyo_utm30lx name="laser" parent="base_link" ros_topic="laser/scan" update_rate="40" ray_count="1081" min_angle="-135" max_angle="135">
-    <origin xyz="0.0 0.0 0.1" rpy="0 0 ${M_PI/4}"/>
+    <origin xyz="0.1 0.1 0.0" rpy="0 0 ${M_PI/4}"/>
   </xacro:hokuyo_utm30lx>
 </robot>

File: mrsl_quadrotor_description/urdf/sensors/hokuyo_utm30lx.urdf.xacro (robot description, xacro)
@@ -1,101 +1,54 @@
 <?xml version="1.0"?>
 <robot xmlns:xacro="http://ros.org/wiki/xacro">
-    <xacro:property name="M_PI" value="3.1415926535897931" />
-    <xacro:macro name="hokuyo_utm30lx_model" params="name parent *origin">
-      <joint name="${name}_joint" type="fixed">
-        <xacro:insert_block name="origin" />
-        <parent link="${parent}"/>
-        <child link="${name}_frame"/>
-      </joint>
-      <link name="${name}_frame">
-        <inertial>
-          <mass value="0.000" />
-          <origin xyz="0 0 0" rpy="0 0 0" />
-          <inertia ixx="2.632e-4" ixy="0" ixz="0" iyy="2.632e-4" iyz="0" izz="1.62e-4" />
-        </inertial>
-        <visual>
-          <origin xyz="0 0 0.0" rpy="0 0 0" />
-          <geometry>
-            <mesh filename="package://mrsl_models/models/sensors/hokuyo_utm_30lx/utm_30lx.dae"/>
+  <xacro:property name="M_PI" value="3.1415926535897931" />
+  <xacro:macro name="hokuyo_utm30lx" params="name parent *origin ros_topic update_rate ray_count min_angle max_angle">
+    <link name="${name}_frame">
+      <inertial>
+        <mass value="0.001" />
+        <origin xyz="0 0 0" rpy="0 0 0" />
+        <inertia ixx="2.632e-4" ixy="0" ixz="0" iyy="2.632e-4" iyz="0" izz="1.62e-4" />
+      </inertial>
+      <visual>
+        <origin xyz="0 0 0" rpy="0 0 0" />
+        <geometry>
+          <mesh filename="package://mrsl_models/models/sensors/hokuyo_utm_30lx/utm_30lx.dae"/>
         </geometry>
-        </visual>
-        <collision>
-          <origin xyz="0 0 0.0" rpy="0 0 0" />
-          <geometry>
-            <!--<box size="0.058 0.058 0.087" />-->
-            <mesh filename="package://mrsl_models/models/sensors/hokuyo_utm_30lx/utm_30lx.stl"/>
-        </geometry>
-        </collision>
-      </link>
-    </xacro:macro>
-    <xacro:macro name="hokuyo_utm30lx" params="name parent *origin ros_topic update_rate ray_count min_angle max_angle">
-      <xacro:hokuyo_utm30lx_model name="${name}" parent="${parent}">
-        <xacro:insert_block name="origin" />
-      </xacro:hokuyo_utm30lx_model>
-      <gazebo reference="${name}_frame">
-        <sensor type="ray" name="${name}">
-          <always_on>true</always_on>
-          <update_rate>${update_rate}</update_rate>
-          <pose>0 0 0 0 0 0</pose>
-          <visualize>false</visualize>
-          <ray>
-            <scan>
-              <horizontal>
-                <samples>${ray_count}</samples>
-                <resolution>1</resolution>
-                <min_angle>${min_angle * M_PI/180}</min_angle>
-                <max_angle>${max_angle * M_PI/180}</max_angle>
-              </horizontal>
-            </scan>
-            <range>
-              <min>0.1</min>
-              <max>30.0</max>
-              <resolution>0.01</resolution>
-            </range>
-          </ray>
-          <plugin name="gazebo_ros_${name}_controller" filename="libgazebo_ros_laser.so">
-            <gaussianNoise>0.005</gaussianNoise>
-            <alwaysOn>true</alwaysOn>
-            <updateRate>${update_rate}</updateRate>
-            <topicName>${ros_topic}</topicName>
-            <frameName>${name}</frameName>
-          </plugin>
-        </sensor>
-      </gazebo>
-    </xacro:macro>
-    <xacro:macro name="hokuyo_utm30lx_gpu" params="name parent *origin ros_topic update_rate ray_count min_angle max_angle">
-      <xacro:hokuyo_utm30lx_model name="${name}" parent="${parent}">
-        <xacro:insert_block name="origin" />
-      </xacro:hokuyo_utm30lx_model>
-      <gazebo reference="${name}_frame">
-        <sensor type="gpu_ray" name="${name}">
-          <always_on>true</always_on>
-          <update_rate>${update_rate}</update_rate>
-          <pose>0 0 0 0 0 0</pose>
-          <visualize>false</visualize>
-          <ray>
-            <scan>
-              <horizontal>
-                <samples>${ray_count}</samples>
-                <resolution>1</resolution>
-                <min_angle>${min_angle * M_PI/180}</min_angle>
-                <max_angle>${max_angle * M_PI/180}</max_angle>
-              </horizontal>
-            </scan>
-            <range>
-              <min>0.3</min>
-              <max>30.0</max>
-              <resolution>0.01</resolution>
-            </range>
-          </ray>
-          <plugin name="gazebo_ros_${name}_controller" filename="libgazebo_ros_gpu_laser.so">
-            <gaussianNoise>0.005</gaussianNoise>
-            <alwaysOn>true</alwaysOn>
-            <updateRate>${update_rate}</updateRate>
-            <topicName>${ros_topic}</topicName>
-            <frameName>${name}_frame</frameName>
-          </plugin>
-        </sensor>
-      </gazebo>
-    </xacro:macro>
+      </visual>
+   </link>
+    <joint name="${name}_joint" type="fixed">
+      <xacro:insert_block name="origin" />
+      <parent link="${parent}"/>
+      <child link="${name}_frame"/>
+    </joint>
+    <gazebo reference="${name}_frame">
+      <sensor type="ray" name="${name}">
+        <always_on>true</always_on>
+        <update_rate>${update_rate}</update_rate>
+        <pose>0 0 0 0 0 0</pose>
+        <visualize>true</visualize>
+        <ray>
+          <scan>
+            <horizontal>
+              <samples>${ray_count}</samples>
+              <resolution>1</resolution>
+              <min_angle>${min_angle * M_PI/180}</min_angle>
+              <max_angle>${max_angle * M_PI/180}</max_angle>
+            </horizontal>
+          </scan>
+          <range>
+            <min>0.1</min>
+            <max>30.0</max>
+            <resolution>0.01</resolution>
+          </range>
+        </ray>
+        <plugin name="gazebo_ros_${name}_controller" filename="libgazebo_ros_laser.so">
+          <gaussianNoise>0.005</gaussianNoise>
+          <alwaysOn>true</alwaysOn>
+          <updateRate>${update_rate}</updateRate>
+          <topicName>${ros_topic}</topicName>
+          <frameName>${name}_frame</frameName>
+        </plugin>
+      </sensor>
+    </gazebo>
+  </xacro:macro>
 </robot>

Commit message: changed tf of laser on pelican_laser model

File: mrsl_quadrotor_description/urdf/pelican_laser/sensors.urdf.xacro (robot description, xacro)
@@ -4,5 +4,5 @@
   <xacro:include filename="$(find mrsl_quadrotor_description)/urdf/sensors/hokuyo_utm30lx.urdf.xacro" />
   <xacro:hokuyo_utm30lx name="laser" parent="base_link" ros_topic="laser/scan" update_rate="40" ray_count="1081" min_angle="-135" max_angle="135">
-    <origin xyz="0.0 0.0 0.2" rpy="0 0 ${M_PI/4}"/>
+    <origin xyz="0.0 0.0 0.2" rpy="0 0 0"/>
   </xacro:hokuyo_utm30lx>
 </robot>
