Commit message: update mobile object plugin, change topic name in msg_to_tf

File: mrsl_quadrotor_description/urdf/mobile_barrel/mobile_barrel.urdf.xacro (robot description, xacro)
@@ -1,12 +1,13 @@
 <?xml version="1.0"?>
-<robot name="mobile_robot" xmlns:xacro="http://ros.org/wiki/xacro">
+<robot name="mobile_object" xmlns:xacro="http://ros.org/wiki/xacro">
   <xacro:property name="pi" value="3.1415926535897931" />
-  <xacro:property name="h" value="3" />
+  <xacro:property name="h" value="2" />
+  <xacro:property name="object" value="barrel" />
   <xacro:property name="mass" value="0.0001" />
   <xacro:property name="ixx" value="0.0001" />
   <xacro:property name="iyy" value="0.0001" />
   <xacro:property name="izz" value="0.0001" />
-  <xacro:macro name="object_base_macro">
-    <link name="base_link">
+  <xacro:macro name="object_base_macro" params="name">
+    <link name="${name}/base_link">
       <inertial>
         <!--mass value="1.477" /-->
@@ -18,14 +19,11 @@
         <origin rpy="0 0 0" xyz="0 0 0"/>
         <geometry>
-          <cylinder length="${h}" radius="0.2"/>
+          <mesh filename="package://mrsl_models/models/${object}/${object}.dae"/>
         </geometry>
-        <material name="red">
-          <color rgba="0.9 0.9 0 1"/>
-        </material>
       </visual>
       <collision>
         <origin rpy="0 0 0" xyz="0 0 0"/>
         <geometry>
-          <cylinder length="${h}" radius="0.2"/>
+          <mesh filename="package://mrsl_models/models/${object}/${object}.dae"/>
         </geometry>
       </collision>
@@ -34,9 +32,14 @@
     <gazebo>
       <!-- Quad Dynamics Plugin -->
-      <plugin name="test" filename="libmrsl_mobile_object.so">
+      <plugin name="mobile_${object}" filename="libmrsl_mobile_object.so">
+        <vx>0.0</vx>
         <vy>1.0</vy>
+        <w>0.0</w>
+        <objectName>${name}</objectName>
+        <topicName>pose</topicName>
+        <updateRate>20.0</updateRate>
     </plugin>
    </gazebo>
   </xacro:macro>
-  <xacro:object_base_macro/>
+  <xacro:object_base_macro name="mobile_${object}"/>
 </robot>
