Commit message: Images Updated

File: mrsl_quadrotor_description/urdf/Falcon4_OS1/Falcon4_OS1.urdf.xacro (robot description, xacro)
@@ -48,5 +48,5 @@
     <origin xyz="0.06 -0.02 0.05" rpy="0 0 0"/>
     </xacro:range_beam_model>
-    <!--Ouster-->
+    <!--Ouster-OS1-->
     <xacro:include filename="$(find mrsl_quadrotor_description)/urdf/sensors/OS1-64.urdf.xacro"/>
     <OS1-64 parent="base_link" name="os1_sensor" hz="10" samples="220">

File: mrsl_quadrotor_description/urdf/sensors/OS1-64.urdf.xacro (robot description, xacro)
@@ -24,5 +24,5 @@
          <origin xyz="0 0 0.0" rpy="0 0 1.5707" />
          <geometry>
-	         <mesh filename="package://ouster_description/meshes/os1_64.dae" />
+	         <mesh filename="package://mrsl_models/models/sensors/OS1-64/os1_64.dae" />
            <!-- <cylinder length="0.073" radius="0.04" /> -->
          </geometry>
