Commit message: Mod-1

File: mrsl_quadrotor_description/urdf/Falcon4/Falcon4.urdf.xacro (robot description, xacro)
@@ -21,7 +21,7 @@
       </visual>
       <collision>
-        <origin xyz="0 0 0" rpy="0 0 0" />
+        <origin xyz="0 0 0.13" rpy="0 0 0" />
         <geometry>
-          <cylinder radius="0.05" length="0.01"/>
+          <cylinder radius="0.52" length="0.2"/>
         </geometry>
       </collision>
@@ -63,4 +63,18 @@
       </plugin>
      </gazebo>
+     <!-- GPS Sensor -->
+     <gazebo>
+        <plugin name="novatel_gps_sim" filename="libhector_gazebo_ros_gps.so">
+        <alwaysOn>1</alwaysOn>
+          <updateRate>10.0</updateRate>
+          <bodyName>base_link</bodyName>
+          <topicName>GPS_Fix</topicName>
+          <velocityTopicName>fix_velocity</velocityTopicName>
+          <drift>5.0 5.0 5.0</drift>
+          <gaussianNoise>0.1 0.1 0.1</gaussianNoise>
+          <velocityDrift>0 0 0</velocityDrift>
+          <velocityGaussianNoise>0.1 0.1 0.1</velocityGaussianNoise>
+      </plugin>
+     </gazebo>
   </xacro:macro>
   <xacro:quadrotor_base_macro/>

File: mrsl_quadrotor_description/urdf/Falcon4_OS1/Falcon4_OS1.urdf.xacro (robot description, xacro)
@@ -22,7 +22,7 @@
       </visual>
       <collision>
-        <origin xyz="0 0 0" rpy="0 0 0" />
+        <origin xyz="0 0 0.13" rpy="0 0 0" />
         <geometry>
-          <cylinder radius="0.05" length="0.01"/>
+          <cylinder radius="0.52" length="0.2"/>
         </geometry>
       </collision>
@@ -50,5 +50,5 @@
     <!--Ouster-OS1-->
     <xacro:include filename="$(find mrsl_quadrotor_description)/urdf/sensors/OS1-64.urdf.xacro"/>
-    <OS1-64 parent="base_link" name="os1_sensor" hz="10" samples="220">
+    <OS1-64 parent="base_link" name="$(arg prefix)" hz="10" samples="220" >
     <origin xyz="0.005 0.01 0.24" rpy="0 0 0" />
     </OS1-64>
@@ -69,4 +69,18 @@
       </plugin>
      </gazebo>
+     <!-- GPS Sensor -->
+     <gazebo>
+        <plugin name="novatel_gps_sim" filename="libhector_gazebo_ros_gps.so">
+        <alwaysOn>1</alwaysOn>
+          <updateRate>10.0</updateRate>
+          <bodyName>base_link</bodyName>
+          <topicName>GPS_Fix</topicName>
+          <velocityTopicName>fix_velocity</velocityTopicName>
+          <drift>5.0 5.0 5.0</drift>
+          <gaussianNoise>0.1 0.1 0.1</gaussianNoise>
+          <velocityDrift>0 0 0</velocityDrift>
+          <velocityGaussianNoise>0.1 0.1 0.1</velocityGaussianNoise>
+      </plugin>
+     </gazebo>
   </xacro:macro>
   <xacro:quadrotor_base_macro/>

File: mrsl_quadrotor_description/urdf/sensors/LidarLite.urdf.xacro (robot description, xacro)
@@ -52,5 +52,5 @@
          <alwaysOn>true</alwaysOn>
          <updateRate>50</updateRate>
-         <topicName>/GroundDist</topicName>
+         <topicName>GroundDist</topicName>
          <frameName>"base_link"</frameName>
          <visualize>true</visualize>

File: mrsl_quadrotor_description/urdf/sensors/OS1-64.urdf.xacro (robot description, xacro)
@@ -2,5 +2,5 @@
 <robot xmlns:xacro="http://www.ros.org/wiki/xacro" name="OS1-64">
   <xacro:property name="M_PI" value="3.1415926535897931" />
-  <xacro:macro name="OS1-64" params="*origin parent:=base_link name:=os1_sensor topic_points:=/os1_cloud_node/points topic_imu:=/os1_cloud_node/imu hz:=10 lasers:=64 samples:=512 min_range:=0.9 max_range:=75.0 noise:=0.008 min_angle:=-${M_PI} max_angle:=${M_PI} lidar_link:=os1_lidar imu_link:=os1_imu vfov_min:=-.26 vfov_max:=.26">
+  <xacro:macro name="OS1-64" params="*origin parent:=base_link name:=os1_sensor topic_points:=os1_cloud_node/points topic_imu:=os1_cloud_node/imu hz:=10 lasers:=64 samples:=512 min_range:=0.9 max_range:=75.0 noise:=0.008 min_angle:=-${M_PI} max_angle:=${M_PI} lidar_link:=os1_lidar imu_link:=os1_imu vfov_min:=-.26 vfov_max:=.26">
     <joint name="${name}_mount_joint" type="fixed">
       <xacro:insert_block name="origin" />
@@ -81,18 +81,18 @@
     </gazebo>
     <!-- IMU -->
-  <gazebo>
-    <plugin name="imu_controller" filename="libhector_gazebo_ros_imu.so">
-      <robotNamespace>/</robotNamespace>
-      <updateRate>100.0</updateRate>
-      <bodyName>${imu_link}</bodyName>
-      <topicName>${topic_imu}</topicName>
-      <accelDrift>0.005 0.005 0.005</accelDrift>
-      <accelGaussianNoise>0.005 0.005 0.005</accelGaussianNoise>
-      <rateDrift>0.005 0.005 0.005 </rateDrift>
-      <rateGaussianNoise>0.005 0.005 0.005 </rateGaussianNoise>
-      <headingDrift>0.005</headingDrift>
-      <headingGaussianNoise>0.005</headingGaussianNoise>
-    </plugin>
-  </gazebo>
+    <gazebo>
+      <plugin name="imu_controller" filename="libhector_gazebo_ros_imu.so">
+        <robotNamespace>/</robotNamespace>
+        <updateRate>100.0</updateRate>
+        <bodyName>${imu_link}</bodyName>
+        <topicName>${topic_imu}</topicName>
+        <accelDrift>0.005 0.005 0.005</accelDrift>
+        <accelGaussianNoise>0.005 0.005 0.005</accelGaussianNoise>
+        <rateDrift>0.005 0.005 0.005 </rateDrift>
+        <rateGaussianNoise>0.005 0.005 0.005 </rateGaussianNoise>
+        <headingDrift>0.005</headingDrift>
+        <headingGaussianNoise>0.005</headingGaussianNoise>
+      </plugin>
+    </gazebo>
   </xacro:macro>
 </robot>

Commit message: Mod - 1.0

File: mrsl_quadrotor_description/urdf/Falcon4/Falcon4.urdf.xacro (robot description, xacro)
@@ -2,6 +2,6 @@
 <robot name="quadrotor" xmlns:xacro="http://ros.org/wiki/xacro">
   <xacro:property name="mass" value="1.5" />
-  <xacro:property name="ixx" value="0.00264" />
-  <xacro:property name="iyy" value="0.00264" />
+  <xacro:property name="ixx" value="0.004" />
+  <xacro:property name="iyy" value="0.004" />
   <xacro:property name="izz" value="0.00496" />
   <!-- Main quadrotor link -->

File: mrsl_quadrotor_description/urdf/Falcon4_OS1/Falcon4_OS1.urdf.xacro (robot description, xacro)
@@ -2,6 +2,6 @@
 <robot name="quadrotor" xmlns:xacro="http://ros.org/wiki/xacro">
   <xacro:property name="mass" value="1.5" />
-  <xacro:property name="ixx" value="0.00264" />
-  <xacro:property name="iyy" value="0.00264" />
+  <xacro:property name="ixx" value="0.004" />
+  <xacro:property name="iyy" value="0.004" />
   <xacro:property name="izz" value="0.00496" />
   <xacro:property name="M_PI" value="3.1415926535897931" />
