Commit message: Falcon4 orientation updated

File: mrsl_quadrotor_description/urdf/falcon4/falcon4.urdf.xacro (robot description, xacro)
@@ -15,5 +15,5 @@
       </inertial>
       <visual>
-        <origin xyz="0 0 0.05" rpy="0 0 0" />
+        <origin xyz="0 0 0.05" rpy="0 0 -${M_PI/2}" />
         <geometry>
           <mesh filename="package://mrsl_models/models/falcon4/falcon4.dae"/>
@@ -31,21 +31,21 @@
     <xacro:include filename="$(find mrsl_quadrotor_description)/urdf/sensors/ovc3_extcam.urdf.xacro" />
     <xacro:stereo_camera name="bonus_right" parent="base_link">
-    <origin xyz="0.084 0.02 0.08" rpy="0 0 0"/>
+    <origin xyz="0.02 -0.084 0.08" rpy="0 0 -${M_PI/2}"/>
     </xacro:stereo_camera>
     <!-- OVC3 Left Side Cam -->
     <xacro:include filename="$(find mrsl_quadrotor_description)/urdf/sensors/ovc3_extcam.urdf.xacro" />
     <xacro:stereo_camera name="bonus_left" parent="base_link">
-    <origin xyz="-0.08 0.02 0.08" rpy="0 0 ${M_PI}"/>
+    <origin xyz="0.02 0.08 0.08" rpy="0 0 ${M_PI/2}"/>
     </xacro:stereo_camera>
     <!-- OVC3 -->
     <xacro:include filename="$(find mrsl_quadrotor_description)/urdf/sensors/ovc3.urdf.xacro" />
     <xacro:stereo_camera name="/" parent="base_link">
-    <origin xyz="0.0 0.1 0.065" rpy="0 0 ${M_PI/2}"/>
+    <origin xyz="0.1 0 0.065" rpy="0 0 0"/>
     </xacro:stereo_camera>
     <!-- Downward facing Lidar -->
-    <xacro:include filename="$(find mrsl_quadrotor_description)/urdf/sensors/lidarlite.urdf.xacro" />
-    <xacro:range_beam_model name="DownFa_Lidar" parent="base_link">
-    <origin xyz="0.06 -0.02 0.05" rpy="0 0 0"/>
-    </xacro:range_beam_model>
+    <xacro:include filename="$(find mrsl_quadrotor_description)/urdf/sensors/range_beam.urdf.xacro" />
+    <xacro:range_beam name="downward_range_beam" parent="base_link" ros_topic="range" update_rate="10">
+      <origin xyz="0 0 0" rpy="0 ${M_PI/2} 0"/>
+    </xacro:range_beam>
     <!-- Plugins -->
     <gazebo>

File: mrsl_quadrotor_description/urdf/falcon4_os1/falcon4_os1.urdf.xacro (robot description, xacro)
@@ -16,5 +16,5 @@
       </inertial>
       <visual>
-        <origin xyz="0 0 0.05" rpy="0 0 0" />
+        <origin xyz="0 0 0.05" rpy="0 0 -${M_PI/2}" />
         <geometry>
           <mesh filename="package://mrsl_models/models/falcon4/falcon4.dae"/>
@@ -32,25 +32,25 @@
     <xacro:include filename="$(find mrsl_quadrotor_description)/urdf/sensors/ovc3_extcam.urdf.xacro" />
     <xacro:stereo_camera name="bonus_right" parent="base_link">
-      <origin xyz="0.084 0.02 0.08" rpy="0 0 0"/>
+      <origin xyz="0.02 -0.084 0.08" rpy="0 0 -${M_PI/2}"/>
     </xacro:stereo_camera>
     <!-- OVC3 Left Side Cam -->
     <xacro:include filename="$(find mrsl_quadrotor_description)/urdf/sensors/ovc3_extcam.urdf.xacro" />
     <xacro:stereo_camera name="bonus_left" parent="base_link">
-      <origin xyz="-0.08 0.02 0.08" rpy="0 0 ${M_PI}"/>
+      <origin xyz="0.02 0.08 0.08" rpy="0 0 ${M_PI/2}"/>
     </xacro:stereo_camera>
     <!-- OVC3 -->
     <xacro:include filename="$(find mrsl_quadrotor_description)/urdf/sensors/ovc3.urdf.xacro" />
     <xacro:stereo_camera name="/" parent="base_link">
-      <origin xyz="0.0 0.1 0.065" rpy="0 0 ${M_PI/2}"/>
+      <origin xyz="0.1 0 0.065" rpy="0 0 0"/>
     </xacro:stereo_camera>
     <!-- Downward facing Lidar -->
-    <xacro:include filename="$(find mrsl_quadrotor_description)/urdf/sensors/lidarlite.urdf.xacro" />
-    <xacro:range_beam_model name="DownFa_Lidar" parent="base_link">
-      <origin xyz="0.06 -0.02 0.05" rpy="0 0 0"/>
-    </xacro:range_beam_model>
+    <xacro:include filename="$(find mrsl_quadrotor_description)/urdf/sensors/range_beam.urdf.xacro" />
+    <xacro:range_beam name="downward_range_beam" parent="base_link" ros_topic="range" update_rate="10">
+      <origin xyz="0 0 -0.02" rpy="0 ${M_PI/2} 0"/>
+    </xacro:range_beam>
     <!--Ouster-OS1-->
     <xacro:include filename="$(find mrsl_quadrotor_description)/urdf/sensors/os1-64.urdf.xacro"/>
     <xacro:OS1-64 parent="base_link" name="os1_sensor" hz="10" samples="220" robot_ns="$(arg robot_ns)" >
-      <origin xyz="0.005 0.01 0.24" rpy="0 0 0" />
+      <origin xyz="0.01 -0.005 0.24" rpy="0 0 0" />
     </xacro:OS1-64>
     <!-- Plugins -->

File: mrsl_quadrotor_description/urdf/sensors/range_beam.urdf.xacro (robot description, xacro)
@@ -17,5 +17,5 @@
           <origin xyz="0 0 0" rpy="0 ${M_PI/2} 0" />
           <geometry>
-            <cylinder radius="0.01" length="0.1"/>
+            <cylinder radius="0.01" length="0.01"/>
        </geometry>
         </visual>

Commit message: OVC3 tf updated

File: mrsl_quadrotor_description/urdf/falcon4/falcon4.urdf.xacro (robot description, xacro)
@@ -40,10 +40,10 @@
     <!-- OVC3 -->
     <xacro:include filename="$(find mrsl_quadrotor_description)/urdf/sensors/ovc3.urdf.xacro" />
-    <xacro:stereo_camera name="/" parent="base_link">
+    <xacro:stereo_camera name="/ovc3" parent="base_link">
     <origin xyz="0.1 0 0.065" rpy="0 0 0"/>
     </xacro:stereo_camera>
     <!-- Downward facing Lidar -->
     <xacro:include filename="$(find mrsl_quadrotor_description)/urdf/sensors/range_beam.urdf.xacro" />
-    <xacro:range_beam name="downward_range_beam" parent="base_link" ros_topic="range" update_rate="10">
+    <xacro:range_beam name="downward_range_beam_frame" parent="base_link" ros_topic="range" update_rate="10">
       <origin xyz="0 0 0" rpy="0 ${M_PI/2} 0"/>
     </xacro:range_beam>

File: mrsl_quadrotor_description/urdf/falcon4_os1/falcon4_os1.urdf.xacro (robot description, xacro)
@@ -41,10 +41,10 @@
     <!-- OVC3 -->
     <xacro:include filename="$(find mrsl_quadrotor_description)/urdf/sensors/ovc3.urdf.xacro" />
-    <xacro:stereo_camera name="/" parent="base_link">
+    <xacro:stereo_camera name="/ovc3" parent="base_link">
       <origin xyz="0.1 0 0.065" rpy="0 0 0"/>
     </xacro:stereo_camera>
     <!-- Downward facing Lidar -->
     <xacro:include filename="$(find mrsl_quadrotor_description)/urdf/sensors/range_beam.urdf.xacro" />
-    <xacro:range_beam name="downward_range_beam" parent="base_link" ros_topic="range" update_rate="10">
+    <xacro:range_beam name="downward_range_beam_frame" parent="base_link" ros_topic="range" update_rate="10">
       <origin xyz="0 0 -0.02" rpy="0 ${M_PI/2} 0"/>
     </xacro:range_beam>
@@ -69,8 +69,8 @@
         <frameName>world</frameName>
       </plugin>
-     </gazebo>
-     <!-- GPS Sensor -->
-     <gazebo>
-        <plugin name="novatel_gps_sim" filename="libhector_gazebo_ros_gps.so">
+    </gazebo>
+    <!-- GPS Sensor -->
+    <gazebo>
+      <plugin name="novatel_gps_sim" filename="libhector_gazebo_ros_gps.so">
         <alwaysOn>1</alwaysOn>
           <updateRate>10.0</updateRate>
@@ -83,5 +83,5 @@
           <velocityGaussianNoise>0.1 0.1 0.1</velocityGaussianNoise>
       </plugin>
-     </gazebo>
+    </gazebo>
   </xacro:macro>
   <xacro:quadrotor_base_macro/>

File: mrsl_quadrotor_description/urdf/sensors/os1-64.urdf.xacro (robot description, xacro)
@@ -16,5 +16,5 @@
       </inertial>
       <collision name="base_collision">
-         <origin xyz="0 0 0.0365" rpy="0 0 0" />
+         <origin xyz="0 0 0" rpy="0 0 0" />
          <geometry>
  	        <cylinder radius="0.04" length="0.073"/>

File: mrsl_quadrotor_description/urdf/sensors/ovc3.urdf.xacro (robot description, xacro)
@@ -29,4 +29,16 @@
       </visual>
     </link>
+    <joint name="${name}_depth_joint" type="fixed">
+        <origin xyz="0.002 0.06 -0.005" rpy="0 0 0" />
+        <parent link="${name}_link" />
+        <child link="${name}_depth_frame"/>
+      </joint>
+      <link name="${name}_depth_frame"/>
+      <joint name="${name}_depth_optical_joint" type="fixed">
+        <origin xyz="0 0 0" rpy="${-M_PI/2} 0.0 ${-M_PI/2}" />
+        <parent link="${name}_depth_frame" />
+        <child link="${name}_depth_optical_frame"/>
+      </joint>
+      <link name="${name}_depth_optical_frame"/>
     <!-- camera -->
     <gazebo reference="${name}_link">

File: mrsl_quadrotor_description/urdf/sensors/ovc3_extcam.urdf.xacro (robot description, xacro)
@@ -29,4 +29,16 @@
       </visual>
     </link>
+    <joint name="${name}_depth_joint" type="fixed">
+        <origin xyz="0.002 0.06 -0.004" rpy="0 0 0" />
+        <parent link="${name}_link" />
+        <child link="${name}_depth_frame"/>
+      </joint>
+      <link name="${name}_depth_frame"/>
+      <joint name="${name}_depth_optical_joint" type="fixed">
+        <origin xyz="0 0 0" rpy="${-M_PI/2} 0.0 ${-M_PI/2}" />
+        <parent link="${name}_depth_frame" />
+        <child link="${name}_depth_optical_frame"/>
+      </joint>
+      <link name="${name}_depth_optical_frame"/>
     <!-- camera -->
     <gazebo reference="${name}_link">
