Commit message: add option to change frame_id of gazebo topics, fix fla models, add tf publisher

File: mrsl_quadrotor_description/urdf/dragon_ddk/camera.urdf.xacro (robot description, xacro)
@@ -2,5 +2,5 @@
 <robot xmlns:xacro="http://ros.org/wiki/xacro">
   <xacro:property name="M_PI" value="3.1415926535897931" />
-  <xacro:macro name="monocular_camera" params="name parent *origin">
+  <xacro:macro name="monocular_camera" params="name parent frame_prefix *origin">
     <joint name="${name}_joint" type="fixed">
       <xacro:insert_block name="origin" />
@@ -48,5 +48,5 @@
           <imageTopicName>image_raw</imageTopicName>
           <cameraInfoTopicName>camera_info</cameraInfoTopicName>
-          <frameName>camera_link</frameName>
+          <frameName>${frame_prefix}camera_link</frameName>
           <hackBaseline>0.07</hackBaseline>
           <distortionK1>0.0</distortionK1>

File: mrsl_quadrotor_description/urdf/dragon_ddk/dragon_ddk.gazebo.xacro (robot description, xacro)
@@ -1,5 +1,6 @@
 <?xml version="1.0"?>
 <robot name="dragon_ddk" xmlns:xacro="http://ros.org/wiki/xacro">
-  <xacro:include filename="$(find mrsl_quadrotor_description)/urdf/dragon_ddk/dragon_ddk_so3.urdf.xacro" />
-  <xacro:include filename="$(find mrsl_quadrotor_description)/urdf/dragon_ddk/sensors.urdf.xacro"/>
+  <xacro:arg name="frame_prefix" default="" />
+  <xacro:include filename="$(find mrsl_quadrotor_description)/urdf/dragon_ddk/dragon_ddk_so3.urdf.xacro"/>
+  <xacro:include filename="$(find mrsl_quadrotor_description)/urdf/dragon_ddk/sensors.urdf.xacro" frame_prefix="$(arg frame_prefix)"/>
 </robot>

File: mrsl_quadrotor_description/urdf/dragon_ddk/rgbd_camera.urdf.xacro (robot description, xacro)
@@ -52,5 +52,5 @@
       <link name="${name}_rgb_optical_frame"/>
     </xacro:macro>
-    <xacro:macro name="rgbd_camera" params="name parent *origin">
+    <xacro:macro name="rgbd_camera" params="name parent frame_prefix *origin">
       <xacro:rgbd_camera_model name="${name}" parent="${parent}">
         <xacro:insert_block name="origin" />
@@ -80,5 +80,5 @@
             <depthImageCameraInfoTopicName>${name}/depth/camera_info</depthImageCameraInfoTopicName>
             <pointCloudTopicName>${name}/depth/points</pointCloudTopicName>
-            <frameName>${name}_depth_optical_frame</frameName>
+            <frameName>${frame_prefix}${name}_depth_optical_frame</frameName>
             <distortion_k1>0.0</distortion_k1>
             <distortion_k2>0.0</distortion_k2>

File: mrsl_quadrotor_description/urdf/dragon_ddk/sensors.urdf.xacro (robot description, xacro)
@@ -1,14 +1,15 @@
 <?xml version="1.0"?>
 <robot xmlns:xacro="http://ros.org/wiki/xacro">
+  <xacro:arg name="frame_prefix" default="" />
   <xacro:include filename="$(find mrsl_quadrotor_description)/urdf/dragon_ddk/camera.urdf.xacro" />
-  <xacro:monocular_camera name="dfc_camera" parent="dfc">
+  <xacro:monocular_camera name="dfc_camera" parent="dfc" frame_prefix="$(arg frame_prefix)">
     <origin xyz="0.0 0.0 0.0" rpy="${M_PI} -${M_PI/2} -${M_PI/2}"/>
   </xacro:monocular_camera>
   <xacro:include filename="$(find mrsl_quadrotor_description)/urdf/dragon_ddk/stereo_camera.urdf.xacro" />
-  <xacro:stereo_camera name="stereo" parent="left_stereo">
+  <xacro:stereo_camera name="stereo" parent="left_stereo" frame_prefix="$(arg frame_prefix)">
     <origin xyz="0.0 0.0 0.0" rpy="0 -${M_PI/2} ${M_PI/2}"/>
   </xacro:stereo_camera>
   <xacro:include filename="$(find mrsl_quadrotor_description)/urdf/dragon_ddk/rgbd_camera.urdf.xacro" />
-  <xacro:rgbd_camera name="rgbd" parent="base_link">
+  <xacro:rgbd_camera name="rgbd" parent="base_link" frame_prefix="$(arg frame_prefix)">
     <origin xyz="0.1 0.0 0.0" rpy="0 0 0"/>
   </xacro:rgbd_camera>
@@ -27,5 +28,5 @@
         <xyzOffset>0 0 0</xyzOffset>
         <rpyOffset>0 0 0</rpyOffset>
-        <frameName>imu</frameName>
+        <frameName>$(arg frame_prefix)imu</frameName>
       </plugin>
       <pose>0 0 0 0 0 0</pose>

File: mrsl_quadrotor_description/urdf/dragon_ddk/stereo_camera.urdf.xacro (robot description, xacro)
@@ -10,5 +10,5 @@
   <xacro:property name="hack_baseline" value="0.08" />
   <xacro:property name="frame_rate" value="15" />
-  <xacro:macro name="stereo_camera" params="name parent *origin">
+  <xacro:macro name="stereo_camera" params="name parent frame_prefix *origin">
     <joint name="${name}_joint" type="fixed">
       <xacro:insert_block name="origin" />
@@ -65,5 +65,5 @@
           <imageTopicName>image_raw</imageTopicName>
           <cameraInfoTopicName>camera_info</cameraInfoTopicName>
-          <frameName>${frame_id}</frameName>
+          <frameName>${frame_prefix}${frame_id}</frameName>
           <hackBaseline>${hack_baseline}</hackBaseline>
           <CxPrime>${(image_width+1)/2}</CxPrime>

File: mrsl_quadrotor_description/urdf/falcon4/falcon4.gazebo.xacro (robot description, xacro)
@@ -1,4 +1,5 @@
 <?xml version="1.0"?>
 <robot name="falcon4" xmlns:xacro="http://ros.org/wiki/xacro">
-  <xacro:include filename="$(find mrsl_quadrotor_description)/urdf/falcon4/falcon4.urdf.xacro" />
+  <xacro:arg name="frame_prefix" default="" />
+  <xacro:include filename="$(find mrsl_quadrotor_description)/urdf/falcon4/falcon4.urdf.xacro" frame_prefix="$(arg frame_prefix)"/>
 </robot>

File: mrsl_quadrotor_description/urdf/falcon4/falcon4.urdf.xacro (robot description, xacro)
@@ -6,6 +6,7 @@
   <xacro:property name="izz" value="0.00496" />
   <xacro:property name="M_PI" value="3.1415926535897931" />
+  <xacro:arg name="frame_prefix" default="" />
   <!-- Main quadrotor link -->
-  <xacro:macro name="quadrotor_base_macro">
+  <xacro:macro name="quadrotor_base_macro" params="frame_prefix">
     <link name="base_link">
       <inertial>
@@ -30,20 +31,20 @@
     <!-- OVC3 Right Side Cam -->
     <xacro:include filename="$(find mrsl_quadrotor_description)/urdf/sensors/ovc3_extcam.urdf.xacro" />
-    <xacro:stereo_camera name="bonus_right" parent="base_link">
+    <xacro:stereo_camera name="bonus_right" parent="base_link" frame_prefix="${frame_prefix}">
     <origin xyz="0.02 -0.084 0.08" rpy="0 0 -${M_PI/2}"/>
     </xacro:stereo_camera>
     <!-- OVC3 Left Side Cam -->
     <xacro:include filename="$(find mrsl_quadrotor_description)/urdf/sensors/ovc3_extcam.urdf.xacro" />
-    <xacro:stereo_camera name="bonus_left" parent="base_link">
+    <xacro:stereo_camera name="bonus_left" parent="base_link" frame_prefix="${frame_prefix}">
     <origin xyz="0.02 0.08 0.08" rpy="0 0 ${M_PI/2}"/>
     </xacro:stereo_camera>
     <!-- OVC3 -->
     <xacro:include filename="$(find mrsl_quadrotor_description)/urdf/sensors/ovc3.urdf.xacro" />
-    <xacro:stereo_camera name="/ovc3" parent="base_link">
+    <xacro:stereo_camera name="/ovc3" parent="base_link" frame_prefix="${frame_prefix}">
     <origin xyz="0.1 0 0.065" rpy="0 0 0"/>
     </xacro:stereo_camera>
     <!-- Downward facing Lidar -->
     <xacro:include filename="$(find mrsl_quadrotor_description)/urdf/sensors/range_beam.urdf.xacro" />
-    <xacro:range_beam name="downward_range_beam_frame" parent="base_link" ros_topic="range" update_rate="10">
+    <xacro:range_beam name="downward_range_beam_frame" parent="base_link" ros_topic="range" update_rate="10" frame_prefix="${frame_prefix}">
       <origin xyz="0 0 0" rpy="0 ${M_PI/2} 0"/>
     </xacro:range_beam>
@@ -79,4 +80,4 @@
      </gazebo>
   </xacro:macro>
-  <xacro:quadrotor_base_macro/>
+  <xacro:quadrotor_base_macro frame_prefix="$(arg frame_prefix)"/>
 </robot>

File: mrsl_quadrotor_description/urdf/falcon4_os1_16_256/falcon4_os1_16_256.gazebo.xacro (robot description, xacro)
@@ -1,4 +1,5 @@
 <?xml version="1.0"?>
 <robot name="falcon4_os1" xmlns:xacro="http://ros.org/wiki/xacro">
-  <xacro:include filename="$(find mrsl_quadrotor_description)/urdf/falcon4_os1_16_256/falcon4_os1_16_256.urdf.xacro" />
+  <xacro:arg name="frame_prefix" default="" />
+  <xacro:include filename="$(find mrsl_quadrotor_description)/urdf/falcon4_os1_16_256/falcon4_os1_16_256.urdf.xacro" frame_prefix="$(arg frame_prefix)"/>
 </robot>

File: mrsl_quadrotor_description/urdf/falcon4_os1_16_256/falcon4_os1_16_256.urdf.xacro (robot description, xacro)
@@ -7,6 +7,7 @@
   <xacro:property name="M_PI" value="3.1415926535897931" />
   <xacro:arg name="robot_ns" default="falcon4"/>
+  <xacro:arg name="frame_prefix" default="" />
   <!-- Main quadrotor link -->
-  <xacro:macro name="quadrotor_base_macro">
+  <xacro:macro name="quadrotor_base_macro" params="frame_prefix">
     <link name="base_link">
       <inertial>
@@ -31,25 +32,25 @@
     <!-- OVC3 Right Side Cam -->
     <xacro:include filename="$(find mrsl_quadrotor_description)/urdf/sensors/ovc3_extcam.urdf.xacro" />
-    <xacro:stereo_camera name="bonus_right" parent="base_link">
+    <xacro:stereo_camera name="bonus_right" parent="base_link" frame_prefix="$(arg frame_prefix)">
       <origin xyz="0.02 -0.084 0.08" rpy="0 0 -${M_PI/2}"/>
     </xacro:stereo_camera>
     <!-- OVC3 Left Side Cam -->
     <xacro:include filename="$(find mrsl_quadrotor_description)/urdf/sensors/ovc3_extcam.urdf.xacro" />
-    <xacro:stereo_camera name="bonus_left" parent="base_link">
+    <xacro:stereo_camera name="bonus_left" parent="base_link" frame_prefix="$(arg frame_prefix)">
       <origin xyz="0.02 0.08 0.08" rpy="0 0 ${M_PI/2}"/>
     </xacro:stereo_camera>
     <!-- OVC3 -->
     <xacro:include filename="$(find mrsl_quadrotor_description)/urdf/sensors/ovc3.urdf.xacro" />
-    <xacro:stereo_camera name="/ovc3" parent="base_link">
+    <xacro:stereo_camera name="/ovc3" parent="base_link" frame_prefix="$(arg frame_prefix)">
       <origin xyz="0.1 0 0.065" rpy="0 0 0"/>
     </xacro:stereo_camera>
     <!-- Downward facing Lidar -->
     <xacro:include filename="$(find mrsl_quadrotor_description)/urdf/sensors/range_beam.urdf.xacro" />
-    <xacro:range_beam name="downward_range_beam_frame" parent="base_link" ros_topic="range" update_rate="10">
+    <xacro:range_beam name="downward_range_beam_frame" parent="base_link" ros_topic="range" update_rate="10" frame_prefix="$(arg frame_prefix)">
       <origin xyz="0 0 -0.02" rpy="0 ${M_PI/2} 0"/>
     </xacro:range_beam>
     <!--Ouster-OS1, hz is frequency, lasers are vertical resolution, samples are horizontal resolution-->
     <xacro:include filename="$(find mrsl_quadrotor_description)/urdf/sensors/os1-64.urdf.xacro"/>
-    <xacro:OS1-64 parent="base_link" name="os1_sensor" hz="5" lasers="16" samples="256" robot_ns="$(arg robot_ns)" >
+    <xacro:OS1-64 parent="base_link" name="os1_sensor" hz="5" lasers="16" samples="256" robot_ns="$(arg robot_ns)" frame_prefix="$(arg frame_prefix)">
       <origin xyz="0.01 -0.005 0.24" rpy="0 0 0" />
     </xacro:OS1-64>
@@ -85,4 +86,4 @@
     </gazebo>
   </xacro:macro>
-  <xacro:quadrotor_base_macro/>
+  <xacro:quadrotor_base_macro frame_prefix="$(arg frame_prefix)"/>
 </robot>

File: mrsl_quadrotor_description/urdf/falcon4_os1_64_512/falcon4_os1_64_512.gazebo.xacro (robot description, xacro)
@@ -1,4 +1,5 @@
 <?xml version="1.0"?>
 <robot name="falcon4_os1" xmlns:xacro="http://ros.org/wiki/xacro">
-  <xacro:include filename="$(find mrsl_quadrotor_description)/urdf/falcon4_os1_64_512/falcon4_os1_64_512.urdf.xacro" />
+  <xacro:arg name="frame_prefix" default="" />
+  <xacro:include filename="$(find mrsl_quadrotor_description)/urdf/falcon4_os1_64_512/falcon4_os1_64_512.urdf.xacro" frame_prefix="$(arg frame_prefix)"/>
 </robot>

File: mrsl_quadrotor_description/urdf/falcon4_os1_64_512/falcon4_os1_64_512.urdf.xacro (robot description, xacro)
@@ -7,6 +7,7 @@
   <xacro:property name="M_PI" value="3.1415926535897931" />
   <xacro:arg name="robot_ns" default="falcon4"/>
+  <xacro:arg name="frame_prefix" default="" />
   <!-- Main quadrotor link -->
-  <xacro:macro name="quadrotor_base_macro">
+  <xacro:macro name="quadrotor_base_macro" params="frame_prefix">
     <link name="base_link">
       <inertial>
@@ -31,25 +32,25 @@
     <!-- OVC3 Right Side Cam -->
     <xacro:include filename="$(find mrsl_quadrotor_description)/urdf/sensors/ovc3_extcam.urdf.xacro" />
-    <xacro:stereo_camera name="bonus_right" parent="base_link">
+    <xacro:stereo_camera name="bonus_right" parent="base_link" frame_prefix="$(arg frame_prefix)">
       <origin xyz="0.02 -0.084 0.08" rpy="0 0 -${M_PI/2}"/>
     </xacro:stereo_camera>
     <!-- OVC3 Left Side Cam -->
     <xacro:include filename="$(find mrsl_quadrotor_description)/urdf/sensors/ovc3_extcam.urdf.xacro" />
-    <xacro:stereo_camera name="bonus_left" parent="base_link">
+    <xacro:stereo_camera name="bonus_left" parent="base_link" frame_prefix="$(arg frame_prefix)">
       <origin xyz="0.02 0.08 0.08" rpy="0 0 ${M_PI/2}"/>
     </xacro:stereo_camera>
     <!-- OVC3 -->
     <xacro:include filename="$(find mrsl_quadrotor_description)/urdf/sensors/ovc3.urdf.xacro" />
-    <xacro:stereo_camera name="/ovc3" parent="base_link">
+    <xacro:stereo_camera name="/ovc3" parent="base_link" frame_prefix="$(arg frame_prefix)">
       <origin xyz="0.1 0 0.065" rpy="0 0 0"/>
     </xacro:stereo_camera>
     <!-- Downward facing Lidar -->
     <xacro:include filename="$(find mrsl_quadrotor_description)/urdf/sensors/range_beam.urdf.xacro" />
-    <xacro:range_beam name="downward_range_beam_frame" parent="base_link" ros_topic="range" update_rate="10">
+    <xacro:range_beam name="downward_range_beam_frame" parent="base_link" ros_topic="range" update_rate="10" frame_prefix="$(arg frame_prefix)">
       <origin xyz="0 0 -0.02" rpy="0 ${M_PI/2} 0"/>
     </xacro:range_beam>
     <!--Ouster-OS1, hz is frequency, lasers are vertical resolution, samples are horizontal resolution-->
     <xacro:include filename="$(find mrsl_quadrotor_description)/urdf/sensors/os1-64.urdf.xacro"/>
-    <xacro:OS1-64 parent="base_link" name="os1_sensor" hz="10" lasers="64" samples="512" robot_ns="$(arg robot_ns)" >
+    <xacro:OS1-64 parent="base_link" name="os1_sensor" hz="10" lasers="64" samples="512" robot_ns="$(arg robot_ns)" frame_prefix="$(arg frame_prefix)" >
       <origin xyz="0.01 -0.005 0.24" rpy="0 0 0" />
     </xacro:OS1-64>
@@ -85,4 +86,4 @@
     </gazebo>
   </xacro:macro>
-  <xacro:quadrotor_base_macro/>
+  <xacro:quadrotor_base_macro frame_prefix="$(arg frame_prefix)"/>
 </robot>

File: mrsl_quadrotor_description/urdf/fla_platform_laser_rgbd/fla_platform_laser_rgbd.gazebo.xacro (robot description, xacro)
@@ -1,5 +1,6 @@
 <?xml version="1.0"?>
 <robot name="fla" xmlns:xacro="http://ros.org/wiki/xacro">
-  <xacro:include filename="$(find mrsl_quadrotor_description)/urdf/fla_platform_laser_rgbd/fla_platform_so3.urdf.xacro" />
-  <xacro:include filename="$(find mrsl_quadrotor_description)/urdf/fla_platform_laser_rgbd/sensors.urdf.xacro"/>
+  <xacro:arg name="frame_prefix" default="" />
+  <xacro:include filename="$(find mrsl_quadrotor_description)/urdf/fla_platform_visual/fla_platform_so3.urdf.xacro" />
+  <xacro:include filename="$(find mrsl_quadrotor_description)/urdf/fla_platform_laser_rgbd/sensors.urdf.xacro" frame_prefix="$(arg frame_prefix)"/>
 </robot>

File: mrsl_quadrotor_description/urdf/fla_platform_laser_rgbd/sensors.urdf.xacro (robot description, xacro)
@@ -1,10 +1,11 @@
 <?xml version="1.0"?>
 <robot xmlns:xacro="http://ros.org/wiki/xacro">
+  <xacro:arg name="frame_prefix" default="" />
   <xacro:include filename="$(find mrsl_quadrotor_description)/urdf/sensors/asus_camera.urdf.xacro" />
-  <xacro:asus_camera name="camera" parent="base_link">
+  <xacro:asus_camera name="camera" parent="base_link" frame_prefix="$(arg frame_prefix)">
     <origin xyz="0.2 0.0 0.2" rpy="${M_PI} 0 0"/>
   </xacro:asus_camera>
   <xacro:include filename="$(find mrsl_quadrotor_description)/urdf/sensors/hokuyo_utm30lx.urdf.xacro" />
-  <xacro:hokuyo_utm30lx name="laser" parent="base_link" ros_topic="laser/scan" update_rate="40" ray_count="1081" min_angle="-135" max_angle="135">
+  <xacro:hokuyo_utm30lx name="laser" parent="base_link" ros_topic="laser/scan" update_rate="40" ray_count="1081" min_angle="-135" max_angle="135" frame_prefix="$(arg frame_prefix)">
     <origin xyz="0.0 0.0 0.35" rpy="0 0 0"/>
   </xacro:hokuyo_utm30lx>

File: mrsl_quadrotor_description/urdf/fla_platform_lidar_3d/fla_platform_lidar_3d.gazebo.xacro (robot description, xacro)
@@ -1,5 +1,6 @@
 <?xml version="1.0"?>
 <robot name="pelican" xmlns:xacro="http://ros.org/wiki/xacro">
-  <xacro:include filename="$(find mrsl_quadrotor_description)/urdf/fla_platform_lidar_3d/fla_platform_so3.urdf.xacro" />
-  <xacro:include filename="$(find mrsl_quadrotor_description)/urdf/fla_platform_lidar_3d/sensors.urdf.xacro"/>
+  <xacro:arg name="frame_prefix" default="" />
+  <xacro:include filename="$(find mrsl_quadrotor_description)/urdf/fla_platform_visual/fla_platform_so3.urdf.xacro" />
+  <xacro:include filename="$(find mrsl_quadrotor_description)/urdf/fla_platform_lidar_3d/sensors.urdf.xacro" frame_prefix="$(arg frame_prefix)"/>
 </robot>

File: mrsl_quadrotor_description/urdf/fla_platform_lidar_3d/sensors.urdf.xacro (robot description, xacro)
@@ -1,6 +1,7 @@
 <?xml version="1.0"?>
 <robot xmlns:xacro="http://ros.org/wiki/xacro">
+  <xacro:arg name="frame_prefix" default="" />
   <xacro:include filename="$(find mrsl_quadrotor_description)/urdf/sensors/hokuyo_utm30lx_rotate.urdf.xacro" />
-  <xacro:hokuyo_utm30lx name="lidar" parent="base_link" ros_topic="laser/scan" update_rate="40" ray_count="1081" min_angle="-135" max_angle="135">
+  <xacro:hokuyo_utm30lx name="lidar" parent="base_link" ros_topic="laser/scan" update_rate="40" ray_count="1081" min_angle="-135" max_angle="135" frame_prefix="$(arg frame_prefix)">
     <origin xyz="0.0 0.0 0.2" rpy="0 0 0"/>
   </xacro:hokuyo_utm30lx>
@@ -18,5 +19,5 @@
 -->
   <xacro:include filename="$(find mrsl_quadrotor_description)/urdf/sensors/camera.urdf.xacro" />
-  <xacro:monocular_camera name="forward" parent="base_link">
+  <xacro:monocular_camera name="forward" parent="base_link" frame_prefix="$(arg frame_prefix)">
     <origin xyz="0.2 0.0 0.0" rpy="0 0 0"/>
   </xacro:monocular_camera>

File: mrsl_quadrotor_description/urdf/fla_platform_rgbd/fla_platform_rgbd.gazebo.xacro (robot description, xacro)
@@ -1,5 +1,6 @@
 <?xml version="1.0"?>
 <robot name="fla" xmlns:xacro="http://ros.org/wiki/xacro">
-  <xacro:include filename="$(find mrsl_quadrotor_description)/urdf/fla_platform_rgbd/fla_platform_so3.urdf.xacro" />
-  <xacro:include filename="$(find mrsl_quadrotor_description)/urdf/fla_platform_rgbd/sensors.urdf.xacro"/>
+  <xacro:arg name="frame_prefix" default="" />
+  <xacro:include filename="$(find mrsl_quadrotor_description)/urdf/fla_platform_visual/fla_platform_so3.urdf.xacro" />
+  <xacro:include filename="$(find mrsl_quadrotor_description)/urdf/fla_platform_rgbd/sensors.urdf.xacro" frame_prefix="$(arg frame_prefix)"/>
 </robot>

File: mrsl_quadrotor_description/urdf/fla_platform_rgbd/sensors.urdf.xacro (robot description, xacro)
@@ -1,6 +1,7 @@
 <?xml version="1.0"?>
 <robot xmlns:xacro="http://ros.org/wiki/xacro">
+  <xacro:arg name="frame_prefix" default="" />
   <xacro:include filename="$(find mrsl_quadrotor_description)/urdf/sensors/asus_camera.urdf.xacro" />
-  <xacro:asus_camera name="camera" parent="base_link">
+  <xacro:asus_camera name="camera" parent="base_link" frame_prefix="$(arg frame_prefix)">
     <origin xyz="0.2 0.0 0.2" rpy="${M_PI} 0 0"/>
   </xacro:asus_camera>

File: mrsl_quadrotor_description/urdf/fla_platform_rgbd_range/fla_platform_rgbd_range.gazebo.xacro (robot description, xacro)
@@ -1,5 +1,6 @@
 <?xml version="1.0"?>
 <robot name="fla" xmlns:xacro="http://ros.org/wiki/xacro">
-  <xacro:include filename="$(find mrsl_quadrotor_description)/urdf/fla_platform_rgbd_range/fla_platform_so3.urdf.xacro" />
-  <xacro:include filename="$(find mrsl_quadrotor_description)/urdf/fla_platform_rgbd_range/sensors.urdf.xacro"/>
+  <xacro:arg name="frame_prefix" default="" />
+  <xacro:include filename="$(find mrsl_quadrotor_description)/urdf/fla_platform_visual/fla_platform_so3.urdf.xacro" />
+  <xacro:include filename="$(find mrsl_quadrotor_description)/urdf/fla_platform_rgbd_range/sensors.urdf.xacro" frame_prefix="$(arg frame_prefix)"/>
 </robot>

File: mrsl_quadrotor_description/urdf/fla_platform_rgbd_range/sensors.urdf.xacro (robot description, xacro)
@@ -1,4 +1,5 @@
 <?xml version="1.0"?>
 <robot xmlns:xacro="http://ros.org/wiki/xacro">
+  <xacro:arg name="frame_prefix" default="" />
   <xacro:include filename="$(find mrsl_quadrotor_description)/urdf/sensors/asus_camera.urdf.xacro" />
   <xacro:asus_camera name="camera" parent="base_link">
@@ -6,5 +7,5 @@
   </xacro:asus_camera>
   <xacro:include filename="$(find mrsl_quadrotor_description)/urdf/sensors/range_beam.urdf.xacro" />
-  <xacro:range_beam name="downward_range_beam" parent="base_link" ros_topic="range" update_rate="10">
+  <xacro:range_beam name="downward_range_beam" parent="base_link" ros_topic="range" update_rate="10" frame_prefix="$(arg frame_prefix)">
     <origin xyz="-0.1 0 -0.05" rpy="0 ${M_PI/2} 0"/>
   </xacro:range_beam>

File: mrsl_quadrotor_description/urdf/fla_platform_velodyne/fla_platform_velodyne.gazebo.xacro (robot description, xacro)
@@ -1,5 +1,6 @@
 <?xml version="1.0"?>
 <robot name="pelican" xmlns:xacro="http://ros.org/wiki/xacro">
-  <xacro:include filename="$(find mrsl_quadrotor_description)/urdf/fla_platform_velodyne/fla_platform_so3.urdf.xacro" />
-  <xacro:include filename="$(find mrsl_quadrotor_description)/urdf/fla_platform_velodyne/sensors.urdf.xacro"/>
+  <xacro:arg name="frame_prefix" default="" />
+  <xacro:include filename="$(find mrsl_quadrotor_description)/urdf/fla_platform_visual/fla_platform_so3.urdf.xacro" />
+  <xacro:include filename="$(find mrsl_quadrotor_description)/urdf/fla_platform_velodyne/sensors.urdf.xacro" frame_prefix="$(arg frame_prefix)"/>
 </robot>
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